File: Power.kicad_sch (KiCad schematic)
At the start: 33 parts, among them U5 RT9068, U6 LMR36510, U7 SY8502, U8 SE8533

Commit message: routed most tracks
Parts:
- added C45: 22u, Capacitor_SMD:C_1206_3216Metric, symbol Device:C_Small
- C36: value 100p -> 1u
- C37: footprint Capacitor_SMD:C_0805_2012Metric -> Capacitor_SMD:C_1206_3216Metric
- D15: footprint Diode_SMD:D_0805_2012Metric -> (none)
- R59, R60: value 1000 -> 1k
Connections:
- net +5V: now also C45.1
- net GND: now also C45.2
Other:
- note added: "???"
- moved on the sheet: D17, R60
Changed lines of the file:
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@@
   (junction (at 113.03 64.77) (diameter 0) (color 0 0 0 0)
   )
+  (junction (at 133.35 64.77) (diameter 0) (color 0 0 0 0)
+  )
   (junction (at 71.12 130.81) (diameter 0) (color 0 0 0 0)
   )
@@
   )
   (junction (at 57.15 60.96) (diameter 0) (color 0 0 0 0)
+  )
+  (junction (at 133.35 76.2) (diameter 0) (color 0 0 0 0)
   )
   (junction (at 124.46 76.2) (diameter 0) (color 0 0 0 0)
@@
     (stroke (width 0) (type default) (color 0 0 0 0))
   )
+  (wire (pts (xy 133.35 64.77) (xy 133.35 68.58))
+    (stroke (width 0) (type default) (color 0 0 0 0))
+  )
   (wire (pts (xy 91.44 130.81) (xy 93.98 130.81))
     (stroke (width 0) (type default) (color 0 0 0 0))
@@
     (stroke (width 0) (type default) (color 0 0 0 0))
   )
-  (wire (pts (xy 124.46 64.77) (xy 129.54 64.77))
+  (wire (pts (xy 124.46 64.77) (xy 133.35 64.77))
     (stroke (width 0) (type default) (color 0 0 0 0))
   )
@@
     (stroke (width 0) (type default) (color 0 0 0 0))
   )
-  (wire (pts (xy 140.97 73.66) (xy 140.97 76.2))
+  (wire (pts (xy 147.32 73.66) (xy 147.32 76.2))
     (stroke (width 0) (type default) (color 0 0 0 0))
   )
@@
     (stroke (width 0) (type default) (color 0 0 0 0))
   )
-  (wire (pts (xy 140.97 64.77) (xy 140.97 66.04))
+  (wire (pts (xy 147.32 64.77) (xy 147.32 66.04))
     (stroke (width 0) (type default) (color 0 0 0 0))
   )
@@
     (stroke (width 0) (type default) (color 0 0 0 0))
   )
+  (wire (pts (xy 133.35 73.66) (xy 133.35 76.2))
+    (stroke (width 0) (type default) (color 0 0 0 0))
+  )
   (wire (pts (xy 113.03 64.77) (xy 118.11 64.77))
     (stroke (width 0) (type default) (color 0 0 0 0))
@@
     (stroke (width 0) (type default) (color 0 0 0 0))
   )
-  (wire (pts (xy 140.97 76.2) (xy 124.46 76.2))
+  (wire (pts (xy 147.32 76.2) (xy 133.35 76.2))
     (stroke (width 0) (type default) (color 0 0 0 0))
   )
@@
     (stroke (width 0) (type default) (color 0 0 0 0))
   )
+  (wire (pts (xy 133.35 64.77) (xy 135.89 64.77))
+    (stroke (width 0) (type default) (color 0 0 0 0))
+  )
   (wire (pts (xy 113.03 78.74) (xy 113.03 81.28))
     (stroke (width 0) (type default) (color 0 0 0 0))
   )
+  (wire (pts (xy 133.35 76.2) (xy 124.46 76.2))
+    (stroke (width 0) (type default) (color 0 0 0 0))
+  )
   (wire (pts (xy 39.37 69.85) (xy 52.07 69.85))
     (stroke (width 0) (type default) (color 0 0 0 0))
@@
     (stroke (width 0) (type default) (color 0 0 0 0))
   )
-  (wire (pts (xy 137.16 64.77) (xy 140.97 64.77))
+  (wire (pts (xy 143.51 64.77) (xy 147.32 64.77))
     (stroke (width 0) (type default) (color 0 0 0 0))
   )
@@
   )
   (text "LMR36510 not available" (at 161.29 41.91 0)
+    (effects (font (size 1.27 1.27)) (justify left bottom))
+  )
+  (text "???\n\n" (at 115.57 92.71 0)
     (effects (font (size 1.27 1.27)) (justify left bottom))
   )
@@
       (effects (font (size 1.27 1.27)) hide)
     )
-    (property "Footprint" "Diode_SMD:D_0805_2012Metric" (id 2) (at 99.06 88.9 0)
+    (property "Footprint" "" (id 2) (at 99.06 88.9 0)
       (effects (font (size 1.27 1.27)) hide)
     )
@@
     (in_bom yes) (on_board yes) (fields_autoplaced)
     (property "Reference" "R59" (id 0) (at 106.68 124.46 90))
-    (property "Value" "1000" (id 1) (at 106.68 127 90))
+    (property "Value" "1k" (id 1) (at 106.68 127 90))
     (property "Footprint" "Resistor_SMD:R_0805_2012Metric" (id 2) (at 106.68 132.588 90)
       (effects (font (size 1.27 1.27)) hide)
@@
     (pin "1")
   )
+  (symbol (lib_id "Device:C_Small") (at 133.35 71.12 0) (unit 1)
+    (in_bom yes) (on_board yes) (fields_autoplaced)
+    (property "Reference" "C45" (id 0) (at 135.89 69.8562 0)
+      (effects (font (size 1.27 1.27)) (justify left))
+    )
+    (property "Value" "22u" (id 1) (at 135.89 72.3962 0)
+      (effects (font (size 1.27 1.27)) (justify left))
+    )
+    (property "Footprint" "Capacitor_SMD:C_1206_3216Metric" (id 2) (at 133.35 71.12 0)
+      (effects (font (size 1.27 1.27)) hide)
+    )
+    (property "Datasheet" "~" (id 3) (at 133.35 71.12 0)
+      (effects (font (size 1.27 1.27)) hide)
+    )
+    (pin "1")
+    (pin "2")
+  )
   (symbol (lib_id "power:GND") (at 238.76 80.01 0) (unit 1)
     (in_bom yes) (on_board yes) (fields_autoplaced)
@@
     (pin "1")
   )
-  (symbol (lib_id "Device:R") (at 133.35 64.77 90) (unit 1)
-    (in_bom yes) (on_board yes) (fields_autoplaced)
-    (property "Reference" "R60" (id 0) (at 133.35 58.42 90))
-    (property "Value" "1000" (id 1) (at 133.35 60.96 90))
-    (property "Footprint" "Resistor_SMD:R_0805_2012Metric" (id 2) (at 133.35 66.548 90)
-      (effects (font (size 1.27 1.27)) hide)
-    )
-    (property "Datasheet" "~" (id 3) (at 133.35 64.77 0)
+  (symbol (lib_id "Device:R") (at 139.7 64.77 90) (unit 1)
+    (in_bom yes) (on_board yes) (fields_autoplaced)
+    (property "Reference" "R60" (id 0) (at 139.7 58.42 90))
+    (property "Value" "1k" (id 1) (at 139.7 60.96 90))
+    (property "Footprint" "Resistor_SMD:R_0805_2012Metric" (id 2) (at 139.7 66.548 90)
+      (effects (font (size 1.27 1.27)) hide)
+    )
+    (property "Datasheet" "~" (id 3) (at 139.7 64.77 0)
       (effects (font (size 1.27 1.27)) hide)
     )
@@
     (pin "9")
   )
-  (symbol (lib_id "Device:LED") (at 140.97 69.85 90) (unit 1)
-    (in_bom yes) (on_board yes) (fields_autoplaced)
-    (property "Reference" "D17" (id 0) (at 144.78 70.1674 90)
+  (symbol (lib_id "Device:LED") (at 147.32 69.85 90) (unit 1)
+    (in_bom yes) (on_board yes) (fields_autoplaced)
+    (property "Reference" "D17" (id 0) (at 151.13 70.1674 90)
       (effects (font (size 1.27 1.27)) (justify right))
     )
-    (property "Value" "RED" (id 1) (at 144.78 72.7074 90)
+    (property "Value" "RED" (id 1) (at 151.13 72.7074 90)
       (effects (font (size 1.27 1.27)) (justify right))
     )
-    (property "Footprint" "LED_SMD:LED_0805_2012Metric" (id 2) (at 140.97 69.85 0)
-      (effects (font (size 1.27 1.27)) hide)
-    )
-    (property "Datasheet" "~" (id 3) (at 140.97 69.85 0)
+    (property "Footprint" "LED_SMD:LED_0805_2012Metric" (id 2) (at 147.32 69.85 0)
+      (effects (font (size 1.27 1.27)) hide)
+    )
+    (property "Datasheet" "~" (id 3) (at 147.32 69.85 0)
       (effects (font (size 1.27 1.27)) hide)
     )
@@
     (in_bom yes) (on_board yes) (fields_autoplaced)
     (property "Reference" "C36" (id 0) (at 91.4463 54.61 90))
-    (property "Value" "100p" (id 1) (at 91.4463 57.15 90))
+    (property "Value" "1u" (id 1) (at 91.4463 57.15 90))
     (property "Footprint" "Capacitor_SMD:C_0805_2012Metric" (id 2) (at 91.44 60.96 0)
       (effects (font (size 1.27 1.27)) hide)
@@
       (effects (font (size 1.27 1.27)) (justify left))
     )
-    (property "Footprint" "Capacitor_SMD:C_0805_2012Metric" (id 2) (at 124.46 71.12 0)
-      (effects (font (size 1.27 1.27)) hide)
-    )
+    (property "Footprint" "Capacitor_SMD:C_1206_3216Metric" (id 2) (at 124.46 71.12 0)
+      (effects (font (size 1.27 1.27)) hide)
+    )

Commit message: new board dimensions
Parts:
- removed C26: 1u, 63V, symbol Device:C
- removed C27: 1u, symbol Device:C
- removed C28: 2.2u, symbol Device:C_Small
- removed C29: 220n, symbol Device:C_Small
- removed C30: 1u, symbol Device:C_Small
- removed C31: 100p, symbol Device:C_Small
- removed C32: 22u, symbol Device:C_Small
- removed L1: 22u, symbol Device:L
- removed R53: 100k, symbol Device:R
- removed R54: 24k9, symbol Device:R
- removed U5: RT9068, symbol FLUX_BMS:RT9068
- removed U6: LMR36510, symbol FLUX_BMS:LMR36510
- C36: renamed from C37; LCSC (none) -> C5672
- C37: renamed from C45; LCSC (none) -> C5672
- D30: renamed from D15; footprint (none) -> Diode_SMD:D_SOD-123
- U6: renamed from U7; LCSC (none) -> c87752
- U7: renamed from U8; LCSC (none) -> c58988
- renumbered C36 to C33, C33 to C34, C34 to C35, C35 to C38, C38 to C39, C39 to C40, D17 to D29, D16 to D31, L2 to L1, R55 to R64, R60 to R65, R56 to R66, R57 to R67, R58 to R68, R59 to R69, TP1 to TP5, TP8 to TP6
Connections:
- no-connect marks 4 -> 0
Other:
- note removed: "LMR36510 not available"
