File: Flux_BMS.kicad_pcb (KiCad board)
At the start: 4 copper layers, 100 x 60 mm, 93 parts, among them J1 Conn_01x13, J2 CAN, Q1 BSS84, Q10 BSS84, Q11 BSS84, Q12 BSS84, Q13 Q_NMOS_SDG, Q14 Q_NMOS_SDG, Q2 BSS84, Q3 BSS84, Q4 BSS84, Q5 BSS84, Q6 BSS84, Q7 BSS84, Q8 BSS84, Q9 BSS84, U1 LTC6811-1, U2 STM32L476RGTx, U3 BQ76200PW, U4 TJA1051T-3, U5 RT9068, X1 8MHz(16pF)

Commit message: update
Parts:
- removed C26: 1u, 63V, Capacitor_SMD:C_1210_3225Metric
- removed C27: 1u, Capacitor_SMD:C_0603_1608Metric
- removed H1, H2: MountingHole_Pad, MountingHole:MountingHole_2.2mm_M2_DIN965_Pad
- removed U5: RT9068, FLUX-BMS:SOP-8_3.9x4.9mm_P1.27mm_with_therma
- added C33: 2.2u/100V, Capacitor_SMD:C_1206_3216Metric, F.Cu at (113.3, 67.5)
- added C34: 220n, Capacitor_SMD:C_0805_2012Metric, F.Cu at (115.5, 68.2)
- added C35: 1u, Capacitor_SMD:C_0805_2012Metric, F.Cu at (126.7, 72.3)
- added C36: 100p, Capacitor_SMD:C_0805_2012Metric, F.Cu at (126.1, 68.5)
- added C37: 22u, Capacitor_SMD:C_0805_2012Metric, F.Cu at (128.1, 68.5)
- added C38: 1u, Capacitor_SMD:C_0805_2012Metric, F.Cu at (143.0, 68.7)
- added C39: 10u, Capacitor_SMD:C_0805_2012Metric, F.Cu at (150.4, 68.7)
- added D10: RED, LED_SMD:LED_0805_2012Metric, F.Cu at (95.8, 132.4)
- added D11: RED, LED_SMD:LED_0805_2012Metric, F.Cu at (96.1, 139.8)
- added D12: RED, LED_SMD:LED_0805_2012Metric, F.Cu at (95.8, 147.8)
- added D13: RED, LED_SMD:LED_0805_2012Metric, F.Cu at (95.0, 67.4)
- added D14: RED, LED_SMD:LED_0805_2012Metric, F.Cu at (95.4, 125.0)
- added D15: D_Schottky, Diode_SMD:D_0805_2012Metric, F.Cu at (130.1, 71.3)
- added D16: RED, LED_SMD:LED_0805_2012Metric, F.Cu at (156.1, 65.3)
- added D17: RED, LED_SMD:LED_0805_2012Metric, F.Cu at (137.1, 65.1)
- added D3: RED, LED_SMD:LED_0805_2012Metric, F.Cu at (94.8, 76.0)
- added D4: RED, LED_SMD:LED_0805_2012Metric, F.Cu at (95.2, 84.0)
- added D5: RED, LED_SMD:LED_0805_2012Metric, F.Cu at (95.0, 92.4)
- added D6: RED, LED_SMD:LED_0805_2012Metric, F.Cu at (95.2, 101.0)
- added D7: RED, LED_SMD:LED_0805_2012Metric, F.Cu at (95.4, 108.6)
- added D8: RED, LED_SMD:LED_0805_2012Metric, F.Cu at (95.3, 116.6)
- added D9: RED, LED_SMD:LED_0805_2012Metric, F.Cu at (94.6, 58.6)
- added J3: Conn_01x02, Connector_AMASS:AMASS_XT60-M_1x02_P7.20mm_Vertical, F.Cu at (134.6, 45.8)
- added J4: Conn_01x05, Connector_PinSocket_2.54mm:PinSocket_1x05_P2.54mm_Vertical, F.Cu at (162.7, 101.4)
- added J5: USB_C_Receptacle_USB2.0, Connector_USB:USB_C_Receptacle_HRO_TYPE-C-31-M-12, F.Cu at (144.3, 146.2)
- added J6: Conn_01x02, Connector_AMASS:AMASS_XT60-M_1x02_P7.20mm_Vertical, F.Cu at (159.6, 45.8)
- added L2: 47u, Inductor_SMD:L_Taiyo-Yuden_NR-50xx, F.Cu at (125.3, 64.0)
- added R41: 470, Resistor_SMD:R_0805_2012Metric, F.Cu at (90.6, 76.0)
- added R42: 470, Resistor_SMD:R_0805_2012Metric, F.Cu at (90.8, 84.0)
- added R43: 470, Resistor_SMD:R_0805_2012Metric, F.Cu at (88.6, 92.4)
- added R44: 470, Resistor_SMD:R_0805_2012Metric, F.Cu at (88.8, 101.0)
- added R45: 470, Resistor_SMD:R_0805_2012Metric, F.Cu at (88.8, 108.6)
- added R46: 470, Resistor_SMD:R_0805_2012Metric, F.Cu at (90.8, 116.6)
- added R47: 470, Resistor_SMD:R_0805_2012Metric, F.Cu at (90.4, 58.6)
- added R48: 470, Resistor_SMD:R_0805_2012Metric, F.Cu at (91.4, 132.2)
- added R49: 470, Resistor_SMD:R_0805_2012Metric, F.Cu at (91.0, 139.8)
- added R50: 470, Resistor_SMD:R_0805_2012Metric, F.Cu at (91.3, 147.6)
- added R51: 470, Resistor_SMD:R_0805_2012Metric, F.Cu at (90.4, 67.2)
- added R52: 470, Resistor_SMD:R_0805_2012Metric, F.Cu at (90.8, 125.0)
- added R55: 100k, Resistor_SMD:R_0805_2012Metric, F.Cu at (114.9, 71.0)
- added R56: 1.6M, Resistor_SMD:R_0805_2012Metric, F.Cu at (114.9, 73.0)
- added R57: 100k, Resistor_SMD:R_0805_2012Metric, F.Cu at (129.9, 75.3)
- added R58: 31k6, Resistor_SMD:R_0805_2012Metric, F.Cu at (123.7, 75.3)
- added R59: 1000, Resistor_SMD:R_0805_2012Metric, F.Cu at (154.1, 65.3)
- added R60: 1000, Resistor_SMD:R_0805_2012Metric, F.Cu at (135.0, 65.1)
- added R65: 5k1, Resistor_SMD:R_0805_2012Metric, F.Cu at (147.9, 139.5)
- added R66: 5k1, Resistor_SMD:R_0805_2012Metric, F.Cu at (140.7, 139.5)
- added R67: R_Shunt, Resistor_SMD:R_Shunt_Vishay_WSKW0612, F.Cu at (135.7, 54.9)
- added TP1: +5V, TestPoint:TestPoint_Pad_D1.5mm, F.Cu at (131.1, 63.1)
- added TP10: TestPoint, FLUX-BMS:PAD, F.Cu at (159.1, 49.6)
- added TP2: CS, TestPoint:TestPoint_Pad_D1.5mm, F.Cu at (124.2, 100.2)
- added TP3: SCK, TestPoint:TestPoint_Pad_D1.5mm, F.Cu at (124.2, 102.8)
- added TP4: SDI, TestPoint:TestPoint_Pad_D1.5mm, F.Cu at (124.2, 88.0)
- added TP5: SDO, TestPoint:TestPoint_Pad_D1.5mm, F.Cu at (124.2, 90.6)
- added TP6: TestPoint, FLUX-BMS:PAD, F.Cu at (127.1, 49.5)
- added TP7: TestPoint, FLUX-BMS:PAD, F.Cu at (134.1, 49.5)
- added TP8: +3V3, TestPoint:TestPoint_Pad_D1.5mm, F.Cu at (155.6, 70.0)
- added TP9: TestPoint, FLUX-BMS:PAD, F.Cu at (152.1, 49.7)
- added U7: SY8502, Package_SO:HSOP-8-1EP_3.9x4.9mm_P1.27mm_EP2.41x3.1mm, F.Cu at (120.5, 70.0)
- added U8: SE8533, Package_TO_SOT_SMD:SOT-89-3, F.Cu at (146.7, 69.6)
- added U9: INA180A3, Package_TO_SOT_SMD:SOT-23-5, F.Cu at (140.9, 55.1)
- C22, C23, C24, C25: footprint Capacitor_SMD:C_0603_1608Metric -> Capacitor_SMD:C_0805_2012Metric
- Q13, Q14: footprint FLUX-BMS:TRANS_DMP2002UPS-13 -> FLUX-BMS:TRANS_DMP2002UPS-13_2
- R39, R40: footprint Resistor_SMD:R_0603_1608Metric -> Resistor_SMD:R_0805_2012Metric
- X1: footprint Crystal:Crystal_SMD_2012-2Pin_2.0x1.2mm -> Crystal:Crystal_SMD_5032-2Pin_5.0x3.2mm
- moved Q10 59.0 mm to (95.8, 144.4), turned to -90 degrees
- moved R28 59.0 mm to (98.6, 144.4)
- moved R29 59.0 mm to (100.6, 144.4)
- moved R30 59.0 mm to (89.2, 144.4)
- moved Q9 54.3 mm to (96.0, 136.6), turned to -90 degrees
- moved R25 54.3 mm to (98.8, 136.6)
- moved R26 54.3 mm to (100.8, 136.6)
- moved R27 54.3 mm to (89.0, 136.6)
- moved Q8 49.6 mm to (95.8, 129.0), turned to -90 degrees
- moved R22 49.6 mm to (98.6, 129.0)
- moved R23 49.6 mm to (100.6, 129.0)
- moved R24 49.6 mm to (89.2, 129.0)
- moved R34 46.9 mm to (98.2, 121.8), turned to 90 degrees
- moved R36 45.9 mm to (88.6, 121.8)
- moved Q12 45.9 mm to (95.4, 121.8), turned to -90 degrees
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Connections:
- Q13 pad 1: Net-(Q13-Pad1) -> V+
- Q14 pad 1: PACK+ -> CHARGER+
- R39 pad 1: Net-(Q13-Pad1) -> V+
- U2 pad 44: unconnected-(U2-Pad44) -> /STM32L476/USB_DM
- U2 pad 45: unconnected-(U2-Pad45) -> /STM32L476/USB_DP
Routing:
- net +3V3: track 102.8 -> 36.6 mm, vias 5 -> 0
- net V-: track 50.7 -> 0.00 mm, vias 1 -> 0
- net /LTC6811/SENSE+_7: track 71.5 -> 32.2 mm, vias 2 -> 0
- net /LTC6811/SENSE+_2: track 18.8 -> 55.6 mm
- net /Charge_control/BQ_PCHG_EN: track 19.0 -> 55.7 mm
- net +5V: track 2.18 -> 36.9 mm
- net /LTC6811/CELL-_1: track 5.52 -> 38.5 mm
- net /LTC6811/SENSE+_12: track 16.0 -> 48.5 mm
- net /LTC6811/BALANCE_2: track 15.7 -> 45.1 mm
- net /Charge_control/BQ_CHG_EN: track 15.5 -> 44.9 mm
- net Net-(Q14-Pad3): track 3.92 -> 33.0 mm
- net /Charge_control/BQ_DSG_EN: track 16.7 -> 45.6 mm
- net /LTC6811/BALANCE_12: track 16.2 -> 44.6 mm
- net /LTC6811/SENSE+_5: track 68.5 -> 40.5 mm, vias 2 -> 0
- net /LTC6811/BALANCE_4: track 8.38 -> 35.2 mm
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- added copper zone on F.Cu, net Net-(C36-Pad2)
Other:
- board size 100 x 60 mm -> 100 x 100 mm
- board text added: "BQ76200"
- board text added: "CAN"
- board text added: "LEDS"
- board text added: "LTC6811"
- board text added: "MCU"
- board text added: "POWER"
- board text added: "USB"

Commit message: routed most tracks
Parts:
- removed D15: D_Schottky, Diode_SMD:D_0805_2012Metric
- removed TP2: CS, TestPoint:TestPoint_Pad_D1.5mm
- removed TP3: SCK, TestPoint:TestPoint_Pad_D1.5mm
- removed TP4: SDI, TestPoint:TestPoint_Pad_D1.5mm
- removed TP5: SDO, TestPoint:TestPoint_Pad_D1.5mm
- added C41: 100n, Capacitor_SMD:C_0805_2012Metric, F.Cu at (170.0, 70.7)
- added C43: 10n, Capacitor_SMD:C_0805_2012Metric, F.Cu at (165.5, 70.4)
- added C44: 1n, Capacitor_SMD:C_0805_2012Metric, F.Cu at (162.7, 139.2)
- added C45: 22u, Capacitor_SMD:C_1206_3216Metric, F.Cu at (149.8, 79.0)
- added J7: Conn_01x05, Connector_JST:JST_PH_B5B-PH-K_1x05_P2.00mm_Vertical, F.Cu at (171.7, 122.0)
- added R74: 100, Resistor_SMD:R_0805_2012Metric, F.Cu at (161.9, 70.3)
- added R75: 56, Resistor_SMD:R_0805_2012Metric, F.Cu at (162.7, 137.2)
- C36: value 100p -> 1u
- C37: footprint Capacitor_SMD:C_0805_2012Metric -> Capacitor_SMD:C_1206_3216Metric
- Q13, Q14: footprint FLUX-BMS:TRANS_DMP2002UPS-13_2 -> FLUX-BMS:TRANS_BSC076N06NS3-G
- R40: value 220 -> 56
- R59, R60: value 1000 -> 1k
- R67: value R_Shunt -> 0.005; footprint Resistor_SMD:R_Shunt_Vishay_WSKW0612 -> Resistor_SMD:R_2512_6332Metric
- U9: value INA180A3 -> INA180A2
- moved U9 62.4 mm to (154.9, 115.8)
- moved J2 35.0 mm to (165.3, 144.3), turned to 180 degrees
- moved R40 26.4 mm to (166.3, 137.2), turned to 180 degrees
- moved C38 25.8 mm to (134.4, 93.0)
- moved C39 25.8 mm to (141.8, 93.0)
- moved D16 25.8 mm to (147.6, 89.7)
- moved R59 25.8 mm to (145.6, 89.7)
- moved TP8 25.8 mm to (147.1, 94.3)
- moved U8 25.8 mm to (138.2, 93.9)
- moved C17 22.2 mm to (132.9, 122.7)
- moved X1 22.2 mm to (144.9, 108.5)
- moved U2 22.2 mm to (142.5, 119.0)
- moved C20 21.9 mm to (137.8, 109.5)
- moved C21 21.9 mm to (137.8, 107.5)
- moved C15 21.8 mm to (142.7, 104.7)
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Connections:
- J5 pad A4: +5V -> unconnected-(J5-PadA4)
- J5 pad A9: +5V -> unconnected-(J5-PadA4)
- J5 pad B4: +5V -> unconnected-(J5-PadA4)
- J5 pad B9: +5V -> unconnected-(J5-PadA4)
- R40 pad 2: /CAN/CAN_L -> Net-(C44-Pad1)
- R67 pad 1: unconnected-(R67-Pad1) -> Net-(R67-Pad1)
- R67 pad 2: unconnected-(R67-Pad2) -> GND
- TP10 pad 1: GND -> Net-(R67-Pad1)
- U2 pad 46: unconnected-(U2-Pad46) -> /STM32L476/SWCLK
- U2 pad 49: unconnected-(U2-Pad49) -> /STM32L476/SWDIO
- U2 pad 58: unconnected-(U2-Pad58) -> /STM32L476/CURRENT_MEASURE_EN
- U2 pad 7: unconnected-(U2-Pad7) -> /STM32L476/NRST
- U3 pad 10: unconnected-(U3-Pad10) -> Net-(R72-Pad1)
- U3 pad 11: unconnected-(U3-Pad11) -> /Charge_control/PACK_V
- U9 pad 2: unconnected-(U9-Pad2) -> GND
- U9 pad 3: unconnected-(U9-Pad3) -> Net-(R67-Pad1)
- U9 pad 4: unconnected-(U9-Pad4) -> GND
- U9 pad 5: unconnected-(U9-Pad5) -> (no net)
Routing:
- net /STM32L476/NRST: track 0.00 -> 59.5 mm
- net /STM32L476/SWCLK: track 0.00 -> 29.7 mm, vias 0 -> 2
- net /CAN/CAN_TX: track 0.00 -> 28.1 mm
- net /STM32L476/LED_RED: track 0.00 -> 27.8 mm
- net /STM32L476/LED_GREEN: track 0.00 -> 26.9 mm
- net /STM32L476/SWDIO: track 0.00 -> 26.3 mm, vias 0 -> 2
- net /LTC6811/LTC_SDO: track 17.8 -> 39.3 mm, vias 0 -> 2
- net /Charge_control/BQ_PMON_EN: track 51.2 -> 72.1 mm
- net /CAN/CAN_RX: track 0.00 -> 19.6 mm
- net /STM32L476/USB_DP: track 0.00 -> 17.6 mm
- net /STM32L476/USB_DM: track 0.00 -> 17.6 mm
- net Net-(Q13-Pad3): track 29.3 -> 45.5 mm, vias 2 -> 0
- net /Charge_control/BQ_CHG_EN: track 44.9 -> 60.2 mm, vias 0 -> 1
- net /Charge_control/PACK_V: track 0.00 -> 15.2 mm
- net /Charge_control/BQ_DSG_EN: track 45.6 -> 59.5 mm, vias 0 -> 1
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- added copper zone on F.Cu, net CHARGER+
- added copper zone on F.Cu, net Net-(Q13-Pad2)
- added copper zone on F.Cu, net V+
Other:
- board text removed: "BQ76200"
- board text removed: "CAN"
- board text removed: "LEDS"
- board text removed: "LTC6811"
- board text removed: "MCU"
- board text removed: "POWER"
- board text removed: "USB"
