File: Flux_BMS.kicad_pcb (KiCad board)
At the start: 4 copper layers, 83 x 65 mm, 235 parts, among them J1 Conn_01x02, J2 Conn_01x02, J3 USB_C_Receptacle_USB2.0, J4 CAN, J5 Conn_01x08, J6 Conn_01x08, J7 Conn_01x05, J8 Conn_01x02, Q14 HYG025N06LS1C2, Q15 HYG025N06LS1C2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

Commit message: before switching to kicad 7
Parts:
- removed J1, J2: Conn_01x02, Connector_AMASS:AMASS_XT60-M_1x02_P7.20mm_Vertical
Routing:
- net +5V: track 109.9 -> 110.7 mm
Other:
- board text added: "-"
- board text added: "B+"
- board text added: "C+"
- board text added: "C0"
- board text added: "C15"
- board text added: "C7"
- board text added: "C8"
- board text added: "CAN"
- board text added: "Flux BMS v0.1 13/01/22"
- board text added: "JLCJLCJLCJLC"
- board text added: "SCL"
- board text added: "SDA"
- board text added: "SWD"
- board text added: "TEMP1"
- board text added: "TEMP2"
- board text added: "USB"

Commit message: V0.2
Parts:
- added C40: 10u, Capacitor_SMD:C_0805_2012Metric, F.Cu at (118.2, 126.9)
- added C51: 220n, Capacitor_SMD:C_0805_2012Metric, F.Cu at (116.3, 131.7)
- added C56: 220n, Capacitor_SMD:C_0805_2012Metric, B.Cu at (112.3, 124.7)
- added C57: 220n, Capacitor_SMD:C_0805_2012Metric, B.Cu at (111.1, 104.2)
- added D30: D, Diode_SMD:D_SOD-323_HandSoldering, F.Cu at (138.8, 112.5)
- added NT3: NetTie_2, NetTie:NetTie-2_SMD_Pad2.0mm, F.Cu at (122.8, 82.9)
- added R69: 1k, Resistor_SMD:R_0805_2012Metric, F.Cu at (116.3, 135.3)
- added R86: 10k, Resistor_SMD:R_0603_1608Metric, F.Cu at (122.0, 124.2)
- added R87: 10k, Resistor_SMD:R_0603_1608Metric, F.Cu at (118.9, 124.2)
- added R88: 1k, Resistor_SMD:R_0805_2012Metric, B.Cu at (112.2, 121.9)
- added R89: 1k, Resistor_SMD:R_0805_2012Metric, B.Cu at (111.1, 101.8)
- added R90: 1k, Resistor_SMD:R_0805_2012Metric, B.Cu at (111.1, 99.4)
- added R91: 1k, Resistor_SMD:R_0805_2012Metric, B.Cu at (112.2, 119.4)
- C35: value 1n2 -> 2n2
- C37: value 47p -> 56p
- D1, D11, D13, D15, D17, D19, D21, D23, D27, D3, D32, D34, D5, D7, D9: footprint Diode_SMD:D_SOD-323 -> Diode_SMD:D_SOD-323_HandSoldering
- L2: value 68u -> 33u
- Q14, Q15: value HYG025N06LS1C2 -> HYG080N10LS1C2
- R13, R17, R21, R25, R29, R33, R37, R41, R45, R49, R5, R55, R72, R76, R9: value 33 -> 100
- R67: value 237k -> 240k
- R83: value 453k -> 316k
- R84: value 49k9 -> 101k
- R85: value 100k -> 41k2
- TP1: value TestPoint -> Battery +
- TP2: value TestPoint -> Battery -
- TP3: value TestPoint -> CHARGER-
- U4: value INA180A2 -> INA181; footprint Package_TO_SOT_SMD:SOT-23-5 -> Package_TO_SOT_SMD:SOT-23-6
- moved C29 25.5 mm to (122.0, 121.0)
- moved TP2 17.2 mm to (124.5, 72.8), turned to 0 degrees
- moved TP3 10.5 mm to (131.6, 72.8), turned to 0 degrees
- moved TP4 9.75 mm to (140.1, 78.9)
- moved NT2 8.15 mm to (130.2, 80.4), turned to 180 degrees
- moved Q15 5.81 mm to (140.2, 82.2), turned to -90 degrees
- moved R61 5.35 mm to (128.1, 80.4), turned to 0 degrees
- moved Q14 4.21 mm to (146.1, 82.2), turned to -90 degrees
- moved NT1 2.86 mm to (126.0, 80.4), turned to 0 degrees
- moved TP1 2.21 mm to (146.2, 78.8)
- moved R2 0.61 mm to (120.2, 126.9)
- moved U4 0.42 mm to (119.6, 121.0)
- moved C49 0.15 mm to (126.6, 112.6)
- moved R82 0.15 mm to (128.6, 112.6)
Connections:
- net /BQ76940/Cell11/SENSE- renamed /BQ76940/VC10B
- net /BQ76940/Cell6/SENSE- renamed /BQ76940/VC5B
- C52 pad 1: V+ -> BAT+
- NT1 pad 1: Net-(NT1-Pad1) -> BAT-
- NT2 pad 1: GND -> /Charge_control/CHG-
- Q14 pad 1: V+ -> BAT+
- Q15 pad 1: CHARGER+ -> CHG+
- R57 pad 1: V+ -> BAT+
- R58 pad 1: CHARGER+ -> BAT+
- R61 pad 1: Net-(NT1-Pad1) -> BAT-
- R61 pad 2: GND -> /Charge_control/CHG-
- TP1 pad 1: V+ -> BAT+
- TP2 pad 1: GND -> BAT-
- TP3 pad 1: Net-(NT1-Pad1) -> /Charge_control/CHG-
- TP4 pad 1: CHARGER+ -> CHG+
- U2 pad 27: unconnected-(U2-Pad27) -> /BQ76940/BQ_BOOT
- U4 pad 5: +3V3 -> /Charge_control/1V65
- U9 pad 2: V+ -> BAT+
- U9 pad 3: V+ -> BAT+
Routing:
- net BAT+: track 0.00 -> 49.7 mm, vias 0 -> 1
- net V+: track 39.1 -> 0.00 mm
- net /BQ76940/VC5X: track 56.2 -> 78.3 mm, vias 1 -> 2
- net /BQ76940/VC10X: track 54.4 -> 71.9 mm, vias 1 -> 2
- net /BQ76940/C0: track 33.6 -> 47.1 mm
- net /BQ76940/TS1: track 6.37 -> 19.0 mm, vias 0 -> 2
- net /BQ76940/VC10B: track 13.6 -> 25.3 mm, vias 0 -> 1
- net /BQ76940/VC5B: track 12.1 -> 22.6 mm, vias 0 -> 1
- net /STM32L476/SWCLK: track 32.0 -> 22.1 mm
- net GND: track 33.8 -> 42.9 mm, vias 21 -> 22
- net Net-(Q15-G): track 5.10 -> 12.8 mm
- net /Charge_control/1V65: track 0.00 -> 7.13 mm
- net Net-(U6-VBUS): track 20.8 -> 14.1 mm, vias 0 -> 2
- net /BQ76940/C5: track 31.9 -> 38.6 mm, vias 0 -> 1
- net /STM32L476/SWDIO: track 26.8 -> 21.1 mm
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- added copper zone on F.Cu, net /Charge_control/CHG-
- added copper zone on F.Cu, net BAT+
- added copper zone on F.Cu, net BAT-
- added copper zone on F.Cu, net CHG+
- removed copper zone on F.Cu, net CHARGER+
- removed copper zone on F.Cu, net Net-(NT1-Pad1)
- removed copper zone on F.Cu, net V+
Other:
- board text added: "BAT+"
- board text added: "BAT-"
- board text added: "CHG+"
- board text added: "CHG-"
- board text added: "Flux BMS v0.2 07/03/22"
- board text removed: "-"
- board text removed: "B+"
- board text removed: "C+"
- board text removed: "Flux BMS v0.1 13/01/22"
