File: BQ76940.kicad_sch (KiCad schematic)
At the start: 34 parts, among them J5 Conn_01x16, U1 BQ76940DBT

Commit message: before meeting
Parts:
- added C33, C34: 1u, Capacitor_SMD:C_0805_2012Metric, symbol Device:C
- added D29: 100V, symbol Device:D
- added Q18: BST82,215, Package_TO_SOT_SMD:SOT-23, symbol Device:Q_NMOS_GSD
- added R64, R66: 100k, Resistor_SMD:R_0805_2012Metric, symbol Device:R
- added R65: 1k, Resistor_SMD:R_0805_2012Metric, symbol Device:R
- C45, C47, C49: footprint (none) -> Capacitor_SMD:C_0805_2012Metric
- R78, R80, R81, R82: footprint (none) -> Resistor_SMD:R_0805_2012Metric
Connections:
- net C15: now also D29.2 (A), R64.2
- net GND: now also U1.42 (SRP), U1.43 (SRN), C33.2, C34.2
- net VC5X: now also R66.1
- net at U1.9 (REGSRC): now also C34.1, Q18.2 (S)
- new net: Q18.1 (G), R66.2
- new net: C33.1, Q18.3 (D), R65.1
- new net: D29.1 (K), R64.1, R65.2

Commit message: almost ready to order
Parts:
- removed J5: Conn_01x16, Connector_JST:JST_XH_S16B-XH-A_1x16_P2.50mm_Horizontal, symbol Connector_Generic:Conn_01x16
- added C31, C38, C39: 10u, Capacitor_SMD:C_0805_2012Metric, symbol Device:C
- added J5, J6: Conn_01x08, Connector_JST:JST_PH_S8B-PH-K_1x08_P2.00mm_Horizontal, symbol Connector_Generic:Conn_01x08
- added R62, R68: 10k, Resistor_SMD:R_0805_2012Metric, symbol Device:R
- D29, D36, D37, D38: footprint (none) -> Diode_SMD:D_SOD-123
- R80, R81: footprint Resistor_SMD:R_0805_2012Metric -> Connector_JST:JST_PH_B2B-PH-K_1x02_P2.00mm_Vertical
Connections:
- net BQ_SCL: now also R68.2
- net BQ_SDA: now also R62.2
- net C0: now also J6.8 (Pin_8)
- net C1: now also J6.7 (Pin_7)
- net C10: now also J5.6 (Pin_6)
- net C11: now also J5.5 (Pin_5)
- net C12: now also J5.4 (Pin_4)
- net C13: now also J5.3 (Pin_3)
- net C14: now also J5.2 (Pin_2)
- net C15: now also J5.1 (Pin_1)
- net C2: now also J6.6 (Pin_6)
- net C3: now also J6.5 (Pin_5)
- net C4: now also J6.4 (Pin_4)
- net C5: now also J6.3 (Pin_3)
- net C6: now also J6.2 (Pin_2)
- net C7: now also J6.1 (Pin_1)
- net C8: now also J5.8 (Pin_8)
- net C9: now also J5.7 (Pin_7)
- net GND: now also C39.2
- net VC10X: now also C31.2, C38.1
- net VC5X: now also C38.2, C39.1
- net BAT renamed VC15X
- net VC15X: now also C31.1
- net Cell1/SENSE- renamed VC0
- net SENSE+_1 renamed VC1
- net SENSE+_10 renamed VC10
- net SENSE+_11 renamed VC11
- net SENSE+_12 renamed VC12
- net SENSE+_13 renamed VC13
- net SENSE+_14 renamed VC14
- net SENSE+_15 renamed VC15
- net SENSE+_2 renamed VC2
- net SENSE+_3 renamed VC3
- net SENSE+_4 renamed VC4
- net SENSE+_5 renamed VC5
- net SENSE+_6 renamed VC6
- net SENSE+_7 renamed VC7
- net SENSE+_8 renamed VC8
- net SENSE+_9 renamed VC9
- new net +3V3: R62.1, R68.1
Other:
- moved on the sheet: D36, D37, D38, R66

Commit message: before switching to kicad 7
Parts:
- C1, C33, C34, C46, C48: LCSC (none) -> C28323
- C43: LCSC (none) -> C338123
- C44, C45, C47, C49: LCSC (none) -> C1779
- D29, D36, D37, D38: LCSC (none) -> C83528
- R62, R68, R82: LCSC (none) -> C17414
- R64, R66: LCSC (none) -> C149504
- R65, R78: LCSC (none) -> C17513
- R79: LCSC (none) -> C2960934
Changed lines of the file:
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@@
+      (effects (font (size 1.27 1.27)) hide)
+    )
+    (property "LCSC" "C83528" (id 4) (at 252.73 101.6 0)
       (effects (font (size 1.27 1.27)) hide)
     )
@@
       (effects (font (size 1.27 1.27)) hide)
     )
+    (property "LCSC" "C1779" (id 4) (at 21.59 72.39 0)
+      (effects (font (size 1.27 1.27)) hide)
+    )
     (pin "1")
     (pin "2")
@@
       (effects (font (size 1.27 1.27)) hide)
     )
+    (property "LCSC" "C1779" (id 4) (at 21.59 114.3 0)
+      (effects (font (size 1.27 1.27)) hide)
+    )
     (pin "1")
     (pin "2")
@@
     )
     (property "Datasheet" "~" (id 3) (at 31.75 104.14 0)
+      (effects (font (size 1.27 1.27)) hide)
+    )
+    (property "LCSC" "C28323" (id 4) (at 31.75 104.14 0)
       (effects (font (size 1.27 1.27)) hide)
     )
@@
       (effects (font (size 1.27 1.27)) hide)
     )
+    (property "LCSC" "C17414" (id 4) (at 21.59 120.65 0)
+      (effects (font (size 1.27 1.27)) hide)
+    )
     (pin "1")
     (pin "2")
@@
       (effects (font (size 1.27 1.27)) hide)
     )
+    (property "LCSC" "C2960934" (id 4) (at 234.95 48.26 0)
+      (effects (font (size 1.27 1.27)) hide)
+    )
     (pin "1")
     (pin "2")
@@
     )
     (property "Datasheet" "~" (id 3) (at 31.75 86.36 0)
+      (effects (font (size 1.27 1.27)) hide)
+    )
+    (property "LCSC" "C28323" (id 4) (at 31.75 86.36 0)
       (effects (font (size 1.27 1.27)) hide)
     )
@@
       (effects (font (size 1.27 1.27)) hide)
     )
+    (property "LCSC" "C17513" (id 4) (at 55.88 31.75 0)
+      (effects (font (size 1.27 1.27)) hide)
+    )
     (pin "1")
     (pin "2")
@@
       (effects (font (size 1.27 1.27)) hide)
     )
+    (property "LCSC" "C149504" (id 4) (at 43.18 43.18 0)
+      (effects (font (size 1.27 1.27)) hide)
+    )
     (pin "1")
     (pin "2")
@@
     )
     (property "Datasheet" "~" (id 3) (at 73.66 45.72 0)
+      (effects (font (size 1.27 1.27)) hide)
+    )
+    (property "LCSC" "C28323" (id 4) (at 73.66 45.72 0)
       (effects (font (size 1.27 1.27)) hide)
     )
@@
       (effects (font (size 1.27 1.27)) hide)
     )
+    (property "LCSC" "C28323" (id 4) (at 49.53 54.61 0)
+      (effects (font (size 1.27 1.27)) hide)
+    )
     (pin "1")
     (pin "2")
@@
     )
     (property "Datasheet" "~" (id 3) (at 247.65 48.26 0)
+      (effects (font (size 1.27 1.27)) hide)
+    )
+    (property "LCSC" "C338123" (id 4) (at 247.65 48.26 0)
       (effects (font (size 1.27 1.27)) hide)
     )
@@
     )
     (property "Datasheet" "~" (id 3) (at 55.88 21.59 0)
+      (effects (font (size 1.27 1.27)) hide)
+    )
+    (property "LCSC" "C83528" (id 4) (at 55.88 21.59 0)
       (effects (font (size 1.27 1.27)) hide)
     )
@@
       (effects (font (size 1.27 1.27)) hide)
     )
+    (property "LCSC" "C28323" (id 4) (at 33.02 127 0)
+      (effects (font (size 1.27 1.27)) hide)
+    )
     (pin "1")
     (pin "2")
@@
     )
     (property "Datasheet" "~" (id 3) (at 44.45 21.59 0)
+      (effects (font (size 1.27 1.27)) hide)
+    )
+    (property "LCSC" "C149504" (id 4) (at 44.45 21.59 0)
       (effects (font (size 1.27 1.27)) hide)
     )
@@
       (effects (font (size 1.27 1.27)) hide)
     )
+    (property "LCSC" "C1779" (id 4) (at 73.66 66.04 0)
+      (effects (font (size 1.27 1.27)) hide)
+    )
     (pin "1")
     (pin "2")
@@
     )
     (property "Datasheet" "~" (id 3) (at 21.59 90.17 0)
+      (effects (font (size 1.27 1.27)) hide)
+    )
+    (property "LCSC" "C1779" (id 4) (at 21.59 90.17 0)
       (effects (font (size 1.27 1.27)) hide)
     )
@@
       (effects (font (size 1.27 1.27)) hide)
     )
+    (property "LCSC" "C17414" (id 4) (at 31.75 54.61 0)
+      (effects (font (size 1.27 1.27)) hide)
+    )
     (pin "1")
     (pin "2")
@@
       (effects (font (size 1.27 1.27)) hide)
     )
+    (property "LCSC" "C83528" (id 4) (at 242.57 101.6 0)
+      (effects (font (size 1.27 1.27)) hide)
+    )
     (pin "1")
     (pin "2")
@@
     )
     (property "Datasheet" "~" (id 3) (at 24.13 54.61 0)
+      (effects (font (size 1.27 1.27)) hide)
+    )
+    (property "LCSC" "C17414" (id 4) (at 24.13 54.61 0)
       (effects (font (size 1.27 1.27)) hide)
     )
@@
       (effects (font (size 1.27 1.27)) hide)
     )
+    (property "LCSC" "C17513" (id 4) (at 128.27 16.51 0)
+      (effects (font (size 1.27 1.27)) hide)
+    )
     (pin "1")
     (pin "2")
@@
       (effects (font (size 1.27 1.27)) hide)
     )
+    (property "LCSC" "C83528" (id 4) (at 232.41 101.6 0)
+      (effects (font (size 1.27 1.27)) hide)
+    )

Commit message: V0.2
Parts:
- added C42 (x3): 220n, Capacitor_SMD:C_0805_2012Metric, symbol Device:C
- added D30: D, Diode_SMD:D_SOD-323_HandSoldering, symbol Device:D
- added R69, R88, R89, R90, R91: 1k, Resistor_SMD:R_0805_2012Metric, symbol Device:R
- C31, C38, C39: LCSC C2932476 -> C440198
- C43: LCSC C338123 -> C1743
- C44, C45, C47, C49: LCSC C1779 -> C440198
Connections:
- net C0: now also R69.2
- net C10: now also R89.2, R90.2
- net C5: now also R88.2, R91.2
- net GND: now also C42.2
- net TS1: now also D30.1 (K)
- net VC0: now also C42.1, R69.1
- net VC10X: now also C42.2, R90.1
- net VC5X: now also C42.2, R91.1
- net Cell11/SENSE- renamed VC10B
- net VC10B: now also C42.1, R89.1
- net Cell6/SENSE- renamed VC5B
- net VC5B: now also C42.1, R88.1
- new net BQ_BOOT: D30.2 (A)
Other:
- moved on the sheet: C31, C38, C39, C43, D36, D37, D38, J5, J6, R78, R79
