File: CAN.kicad_sch (KiCad schematic)
At the start: 6 parts, among them U5 TJA1051T-3

Commit message: almost ready to order
Parts:
- removed C31: 1n, Capacitor_SMD:C_0805_2012Metric, symbol Device:C
- removed R62: 56, Resistor_SMD:R_0805_2012Metric, symbol Device:R
- C30, C32: footprint Capacitor_SMD:C_0805_2012Metric -> Capacitor_SMD:C_0603_1608Metric
- R63: value 56 -> 120; LCSC C422823 -> (none)
Connections:
- net CAN_H: now also R63.1
Other:
- moved on the sheet: R63
Changed lines of the file:
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@@
   (junction (at 93.98 96.52) (diameter 0) (color 0 0 0 0)
   )
-  (junction (at 151.13 93.98) (diameter 0) (color 0 0 0 0)
-  )
   (junction (at 127 71.12) (diameter 0) (color 0 0 0 0)
   )
-  (junction (at 151.13 109.22) (diameter 0) (color 0 0 0 0)
-  )
-  (junction (at 151.13 78.74) (diameter 0) (color 0 0 0 0)
+  (junction (at 151.13 104.14) (diameter 0) (color 0 0 0 0)
+  )
+  (junction (at 151.13 85.09) (diameter 0) (color 0 0 0 0)
   )
   (junction (at 106.68 109.22) (diameter 0) (color 0 0 0 0)
@@
     (stroke (width 0) (type default) (color 0 0 0 0))
   )
-  (wire (pts (xy 151.13 88.9) (xy 151.13 93.98))
-    (stroke (width 0) (type default) (color 0 0 0 0))
-  )
-  (wire (pts (xy 161.29 102.87) (xy 161.29 104.14))
-    (stroke (width 0) (type default) (color 0 0 0 0))
-  )
-  (wire (pts (xy 144.78 78.74) (xy 151.13 78.74))
-    (stroke (width 0) (type default) (color 0 0 0 0))
-  )
-  (wire (pts (xy 144.78 91.44) (xy 144.78 78.74))
+  (wire (pts (xy 151.13 85.09) (xy 151.13 91.44))
+    (stroke (width 0) (type default) (color 0 0 0 0))
+  )
+  (wire (pts (xy 144.78 85.09) (xy 151.13 85.09))
+    (stroke (width 0) (type default) (color 0 0 0 0))
+  )
+  (wire (pts (xy 144.78 91.44) (xy 144.78 85.09))
     (stroke (width 0) (type default) (color 0 0 0 0))
   )
@@
     (stroke (width 0) (type default) (color 0 0 0 0))
   )
-  (wire (pts (xy 151.13 93.98) (xy 161.29 93.98))
-    (stroke (width 0) (type default) (color 0 0 0 0))
-  )
   (wire (pts (xy 93.98 109.22) (xy 93.98 111.76))
     (stroke (width 0) (type default) (color 0 0 0 0))
@@
     (stroke (width 0) (type default) (color 0 0 0 0))
   )
-  (wire (pts (xy 151.13 105.41) (xy 151.13 109.22))
-    (stroke (width 0) (type default) (color 0 0 0 0))
-  )
-  (wire (pts (xy 151.13 93.98) (xy 151.13 97.79))
+  (wire (pts (xy 151.13 99.06) (xy 151.13 104.14))
     (stroke (width 0) (type default) (color 0 0 0 0))
   )
@@
     (stroke (width 0) (type default) (color 0 0 0 0))
   )
-  (wire (pts (xy 144.78 109.22) (xy 151.13 109.22))
+  (wire (pts (xy 144.78 104.14) (xy 151.13 104.14))
     (stroke (width 0) (type default) (color 0 0 0 0))
   )
@@
     (stroke (width 0) (type default) (color 0 0 0 0))
   )
-  (wire (pts (xy 151.13 78.74) (xy 151.13 81.28))
-    (stroke (width 0) (type default) (color 0 0 0 0))
-  )
-  (wire (pts (xy 151.13 109.22) (xy 163.83 109.22))
+  (wire (pts (xy 151.13 104.14) (xy 163.83 104.14))
     (stroke (width 0) (type default) (color 0 0 0 0))
   )
@@
     (stroke (width 0) (type default) (color 0 0 0 0))
   )
-  (wire (pts (xy 151.13 78.74) (xy 162.56 78.74))
-    (stroke (width 0) (type default) (color 0 0 0 0))
-  )
-  (wire (pts (xy 161.29 95.25) (xy 161.29 93.98))
+  (wire (pts (xy 151.13 85.09) (xy 162.56 85.09))
     (stroke (width 0) (type default) (color 0 0 0 0))
   )
@@
     (stroke (width 0) (type default) (color 0 0 0 0))
   )
-  (wire (pts (xy 144.78 96.52) (xy 144.78 109.22))
+  (wire (pts (xy 144.78 96.52) (xy 144.78 104.14))
     (stroke (width 0) (type default) (color 0 0 0 0))
   )
@@
     (effects (font (size 1.27 1.27)) (justify right))
   )
-  (hierarchical_label "CAN_L" (shape input) (at 163.83 109.22 0)
+  (hierarchical_label "CAN_L" (shape input) (at 163.83 104.14 0)
     (effects (font (size 1.27 1.27)) (justify left))
   )
-  (hierarchical_label "CAN_H" (shape input) (at 162.56 78.74 0)
+  (hierarchical_label "CAN_H" (shape input) (at 162.56 85.09 0)
     (effects (font (size 1.27 1.27)) (justify left))
   )
@@
       (effects (font (size 1.27 1.27)) (justify left))
     )
-    (property "Footprint" "Capacitor_SMD:C_0805_2012Metric" (id 2) (at 94.9452 106.68 0)
+    (property "Footprint" "Capacitor_SMD:C_0603_1608Metric" (id 2) (at 94.9452 106.68 0)
       (effects (font (size 1.27 1.27)) hide)
     )
@@
       (effects (font (size 1.27 1.27)) (justify left))
     )
-    (property "Footprint" "Capacitor_SMD:C_0805_2012Metric" (id 2) (at 122.8852 80.01 0)
+    (property "Footprint" "Capacitor_SMD:C_0603_1608Metric" (id 2) (at 122.8852 80.01 0)
       (effects (font (size 1.27 1.27)) hide)
     )
@@
     (pin "1")
     (pin "2")
-  )
-  (symbol (lib_id "power:GND") (at 161.29 104.14 0) (unit 1)
-    (in_bom yes) (on_board yes)
-    (property "Reference" "#PWR032" (id 0) (at 161.29 110.49 0)
-      (effects (font (size 1.27 1.27)) hide)
-    )
-    (property "Value" "GND" (id 1) (at 157.48 106.68 0))
-    (property "Footprint" "" (id 2) (at 161.29 104.14 0)
-      (effects (font (size 1.27 1.27)) hide)
-    )
-    (property "Datasheet" "" (id 3) (at 161.29 104.14 0)
-      (effects (font (size 1.27 1.27)) hide)
-    )
-    (pin "1")
   )
   (symbol (lib_id "power:+3V3") (at 93.98 92.71 0) (unit 1)
@@
     (pin "1")
   )
-  (symbol (lib_id "Device:R") (at 151.13 101.6 0) (unit 1)
-    (in_bom yes) (on_board yes) (fields_autoplaced)
-    (property "Reference" "R63" (id 0) (at 153.67 100.3299 0)
-      (effects (font (size 1.27 1.27)) (justify left))
-    )
-    (property "Value" "56" (id 1) (at 153.67 102.8699 0)
-      (effects (font (size 1.27 1.27)) (justify left))
-    )
-    (property "Footprint" "Resistor_SMD:R_0805_2012Metric" (id 2) (at 149.352 101.6 90)
-      (effects (font (size 1.27 1.27)) hide)
-    )
-    (property "Datasheet" "~" (id 3) (at 151.13 101.6 0)
-      (effects (font (size 1.27 1.27)) hide)
-    )
-    (property "LCSC" "C422823" (id 4) (at 151.13 101.6 0)
-      (effects (font (size 1.27 1.27)) hide)
-    )
-    (pin "1")
-    (pin "2")
-  )
-  (symbol (lib_id "Device:R") (at 151.13 85.09 0) (unit 1)
-    (in_bom yes) (on_board yes) (fields_autoplaced)
-    (property "Reference" "R62" (id 0) (at 153.67 83.8199 0)
-      (effects (font (size 1.27 1.27)) (justify left))
-    )
-    (property "Value" "56" (id 1) (at 153.67 86.3599 0)
-      (effects (font (size 1.27 1.27)) (justify left))
-    )
-    (property "Footprint" "Resistor_SMD:R_0805_2012Metric" (id 2) (at 149.352 85.09 90)
-      (effects (font (size 1.27 1.27)) hide)
-    )
-    (property "Datasheet" "~" (id 3) (at 151.13 85.09 0)
-      (effects (font (size 1.27 1.27)) hide)
-    )
-    (property "LCSC" "C17757" (id 4) (at 151.13 85.09 0)
+  (symbol (lib_id "Device:R") (at 151.13 95.25 0) (unit 1)
+    (in_bom yes) (on_board yes) (fields_autoplaced)
+    (property "Reference" "R63" (id 0) (at 153.67 93.9799 0)
+      (effects (font (size 1.27 1.27)) (justify left))
+    )
+    (property "Value" "120" (id 1) (at 153.67 96.5199 0)
+      (effects (font (size 1.27 1.27)) (justify left))
+    )
+    (property "Footprint" "Resistor_SMD:R_0805_2012Metric" (id 2) (at 149.352 95.25 90)
+      (effects (font (size 1.27 1.27)) hide)
+    )
+    (property "Datasheet" "~" (id 3) (at 151.13 95.25 0)
+      (effects (font (size 1.27 1.27)) hide)
+    )
+    (property "LCSC" "" (id 4) (at 151.13 95.25 0)
       (effects (font (size 1.27 1.27)) hide)
     )
@@
     (pin "1")
   )
-  (symbol (lib_id "Device:C") (at 161.29 99.06 0) (unit 1)
-    (in_bom yes) (on_board yes) (fields_autoplaced)
-    (property "Reference" "C31" (id 0) (at 165.1 97.7899 0)
-      (effects (font (size 1.27 1.27)) (justify left))
-    )
-    (property "Value" "1n" (id 1) (at 165.1 100.3299 0)
-      (effects (font (size 1.27 1.27)) (justify left))
-    )
-    (property "Footprint" "Capacitor_SMD:C_0805_2012Metric" (id 2) (at 162.2552 102.87 0)
-      (effects (font (size 1.27 1.27)) hide)
-    )
-    (property "Datasheet" "~" (id 3) (at 161.29 99.06 0)
-      (effects (font (size 1.27 1.27)) hide)
-    )
-    (property "LCSC" "C440004" (id 4) (at 161.29 99.06 0)
-      (effects (font (size 1.27 1.27)) hide)
-    )
-    (pin "1")
-    (pin "2")
-  )
 )

Commit message: before switching to kicad 7
Parts:
- C30, C32: LCSC (none) -> C57895
- R63: LCSC (none) -> C17437
Changed lines of the file:
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@@
+      (effects (font (size 1.27 1.27)) hide)
+    )
+    (property "LCSC" "C57895" (id 4) (at 93.98 102.87 0)
       (effects (font (size 1.27 1.27)) hide)
     )
@@
       (effects (font (size 1.27 1.27)) hide)
     )
+    (property "LCSC" "C57895" (id 4) (at 121.92 76.2 0)
+      (effects (font (size 1.27 1.27)) hide)
+    )
     (pin "1")
     (pin "2")
@@
       (effects (font (size 1.27 1.27)) hide)
     )
-    (property "LCSC" "" (id 4) (at 151.13 95.25 0)
+    (property "LCSC" "C17437" (id 4) (at 151.13 95.25 0)
       (effects (font (size 1.27 1.27)) hide)
     )

Commit message: V0.2
Parts:
- C30, C32: LCSC C57895 -> C23630
