File: Flux_BMS.kicad_sch (KiCad schematic)
At the start: 10 parts, among them J2 CAN, J3 Conn_01x02, J5 USB_C_Receptacle_USB2.0, J6 Conn_01x02

Commit message: routed most tracks
Parts:
- removed TP10, TP9: TestPoint, FLUX-BMS:PAD, symbol Connector:TestPoint
Connections:
- net +5V: no longer names the net of J5.A4 (VBUS), J5.A9 (VBUS), J5.B4 (VBUS), J5.B9 (VBUS)
- no-connect marks 2 -> 4

Commit message: new board dimensions
Parts:
- added H1, H2, H3, H4: MountingHole, MountingHole:MountingHole_3.2mm_M3, symbol Mechanical:MountingHole
- J3: renamed from J5; LCSC (none) -> C2927038
- renumbered J3 to J1, J6 to J2, J2 to J4, R65 to R1, R66 to R2, TP6 to TP1, TP7 to TP2
Other:
- sheet LTC6811 renamed BQ76940
- sheet BQ76940: file LTC6811.kicad_sch -> BQ76940.kicad_sch

Commit message: placed bleed resistors
Connections:
- no-connect marks 4 -> 3
Other:
- sheet Power: file Power.kicad_sch -> LM5164.kicad_sch

Commit message: before meeting
Parts:
- added U6: USBLC6-2SC6, Package_TO_SOT_SMD:SOT-23-6, symbol Power_Protection:USBLC6-2SC6
Connections:
- net GND: now also U6.2 (GND)
- net STM32L476/USB_DM: now also U6.4 (I/O2); no longer J3.A7 (D-), J3.B7 (D-)
- net STM32L476/USB_DP: now also U6.3 (I/O2); no longer J3.A6 (D+), J3.B6 (D+)
- net at J3.A4 (VBUS), J3.A9 (VBUS), J3.B4 (VBUS)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: now also U6.5 (VBUS)
- new net: J3.A6 (D+), J3.B6 (D+), U6.1 (I/O1)
- new net: J3.A7 (D-), J3.B7 (D-), U6.6 (I/O1)
- no-connect marks 3 -> 2
Changed lines of the file:
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@@
 (kicad_sch (version 20211123) (generator eeschema)
   (paper "A4")
+  (junction (at 55.88 46.99) (diameter 0) (color 0 0 0 0)
+  )
   (junction (at 58.42 59.69) (diameter 0) (color 0 0 0 0)
   )
-  (junction (at 55.88 46.99) (diameter 0) (color 0 0 0 0)
-  )
   (junction (at 55.88 41.91) (diameter 0) (color 0 0 0 0)
   )
   (junction (at 38.1 68.58) (diameter 0) (color 0 0 0 0)
   )
-  (no_connect (at 53.34 29.21))
   (no_connect (at 53.34 57.15))
   (no_connect (at 53.34 59.69))
-  (wire (pts (xy 55.88 41.91) (xy 105.41 41.91))
-    (stroke (width 0) (type default) (color 0 0 0 0))
-  )
   (wire (pts (xy 53.34 41.91) (xy 55.88 41.91))
     (stroke (width 0) (type default) (color 0 0 0 0))
@@
     (stroke (width 0) (type default) (color 0 0 0 0))
   )
+  (wire (pts (xy 85.09 54.61) (xy 85.09 55.88))
+    (stroke (width 0) (type default) (color 0 0 0 0))
+  )
   (wire (pts (xy 274.32 33.02) (xy 274.32 46.99))
     (stroke (width 0) (type default) (color 0 0 0 0))
   )
+  (wire (pts (xy 95.25 41.91) (xy 105.41 41.91))
+    (stroke (width 0) (type default) (color 0 0 0 0))
+  )
   (wire (pts (xy 95.25 90.17) (xy 105.41 90.17))
     (stroke (width 0) (type default) (color 0 0 0 0))
@@
     (stroke (width 0) (type default) (color 0 0 0 0))
   )
+  (wire (pts (xy 85.09 29.21) (xy 85.09 34.29))
+    (stroke (width 0) (type default) (color 0 0 0 0))
+  )
   (wire (pts (xy 102.87 129.54) (xy 96.52 129.54))
     (stroke (width 0) (type default) (color 0 0 0 0))
@@
     (stroke (width 0) (type default) (color 0 0 0 0))
   )
+  (wire (pts (xy 53.34 29.21) (xy 85.09 29.21))
+    (stroke (width 0) (type default) (color 0 0 0 0))
+  )
   (wire (pts (xy 267.97 33.02) (xy 274.32 33.02))
     (stroke (width 0) (type default) (color 0 0 0 0))
@@
     (stroke (width 0) (type default) (color 0 0 0 0))
   )
+  (wire (pts (xy 55.88 46.99) (xy 74.93 46.99))
+    (stroke (width 0) (type default) (color 0 0 0 0))
+  )
   (wire (pts (xy 267.97 33.02) (xy 267.97 36.83))
     (stroke (width 0) (type default) (color 0 0 0 0))
@@
     (stroke (width 0) (type default) (color 0 0 0 0))
   )
+  (wire (pts (xy 55.88 41.91) (xy 74.93 41.91))
+    (stroke (width 0) (type default) (color 0 0 0 0))
+  )
+  (wire (pts (xy 95.25 46.99) (xy 105.41 46.99))
+    (stroke (width 0) (type default) (color 0 0 0 0))
+  )
   (wire (pts (xy 154.94 85.09) (xy 163.83 85.09))
-    (stroke (width 0) (type default) (color 0 0 0 0))
-  )
-  (wire (pts (xy 55.88 46.99) (xy 105.41 46.99))
     (stroke (width 0) (type default) (color 0 0 0 0))
   )
@@
     )
   )
+  (symbol (lib_id "power:GND") (at 85.09 55.88 0) (unit 1)
+    (in_bom yes) (on_board yes) (fields_autoplaced)
+    (property "Reference" "#PWR?" (id 0) (at 85.09 62.23 0)
+      (effects (font (size 1.27 1.27)) hide)
+    )
+    (property "Value" "GND" (id 1) (at 85.09 60.96 0))
+    (property "Footprint" "" (id 2) (at 85.09 55.88 0)
+      (effects (font (size 1.27 1.27)) hide)
+    )
+    (property "Datasheet" "" (id 3) (at 85.09 55.88 0)
+      (effects (font (size 1.27 1.27)) hide)
+    )
+    (pin "1")
+  )
   (symbol (lib_id "Connector:TestPoint") (at 267.97 36.83 180) (unit 1)
     (in_bom yes) (on_board yes)
@@
     )
     (pin "1")
+  )
+  (symbol (lib_id "Power_Protection:USBLC6-2SC6") (at 85.09 44.45 0) (unit 1)
+    (in_bom yes) (on_board yes) (fields_autoplaced)
+    (property "Reference" "U6" (id 0) (at 87.8587 31.75 0)
+      (effects (font (size 1.27 1.27)) (justify left))
+    )
+    (property "Value" "USBLC6-2SC6" (id 1) (at 87.8587 34.29 0)
+      (effects (font (size 1.27 1.27)) (justify left))
+    )
+    (property "Footprint" "Package_TO_SOT_SMD:SOT-23-6" (id 2) (at 85.09 57.15 0)
+      (effects (font (size 1.27 1.27)) hide)
+    )
+    (property "Datasheet" "https://www.st.com/resource/en/datasheet/usblc6-2.pdf" (id 3) (at 90.17 35.56 0)
+      (effects (font (size 1.27 1.27)) hide)
+    )
+    (property "LCSC" "C2827654" (id 4) (at 85.09 44.45 0)
+      (effects (font (size 1.27 1.27)) hide)
+    )
+    (pin "1")
+    (pin "2")
+    (pin "3")
+    (pin "4")
+    (pin "5")
+    (pin "6")
   )
   (symbol (lib_id "Connector_Generic:Conn_01x02") (at 31.75 123.19 0) (mirror y) (unit 1)
@@
       (reference "#PWR0110") (unit 1) (value "GND") (footprint "")
     )
+    (path "/8f77faa8-2d4a-4750-9ffd-4f5c63ff8509/0aaea52c-1ecf-4025-bd94-53d0c88756fa"
+      (reference "#PWR0111") (unit 1) (value "GND") (footprint "")
+    )
+    (path "/8f77faa8-2d4a-4750-9ffd-4f5c63ff8509/607c8050-92a9-4172-8c7c-95c61150f0a2"
+      (reference "#PWR0112") (unit 1) (value "GND") (footprint "")
+    )
+    (path "/10795709-c265-4ae8-a1a4-1045415b2bf7"
+      (reference "#PWR?") (unit 1) (value "GND") (footprint "")
+    )
     (path "/8f77faa8-2d4a-4750-9ffd-4f5c63ff8509/7b9bc166-f185-4f58-a2e5-50627897da34"
       (reference "C1") (unit 1) (value "1u") (footprint "Capacitor_SMD:C_0805_2012Metric")
@@
       (reference "C32") (unit 1) (value "2u2") (footprint "Capacitor_SMD:C_0805_2012Metric")
     )
+    (path "/8f77faa8-2d4a-4750-9ffd-4f5c63ff8509/4c16054a-2daf-4f91-9807-fc1cca5ba7c8"
+      (reference "C33") (unit 1) (value "1u") (footprint "Capacitor_SMD:C_0805_2012Metric")
+    )
+    (path "/8f77faa8-2d4a-4750-9ffd-4f5c63ff8509/56de294e-d30d-4609-8e10-fb2ae4973b4b"
+      (reference "C34") (unit 1) (value "1u") (footprint "Capacitor_SMD:C_0805_2012Metric")
+    )
     (path "/8f77faa8-2d4a-4750-9ffd-4f5c63ff8509/497a26da-8b1e-4bb2-bcf1-f7f1ed65cd77/4184a390-20bb-4b6a-ba29-e1d6e768cba4"
       (reference "C41") (unit 1) (value "~") (footprint "Capacitor_SMD:C_0805_2012Metric")
@@
     )
     (path "/8f77faa8-2d4a-4750-9ffd-4f5c63ff8509/0a4d1b7c-3666-4f38-808a-87c8b7d79b23"
-      (reference "C45") (unit 1) (value "4u7") (footprint "")
+      (reference "C45") (unit 1) (value "4u7") (footprint "Capacitor_SMD:C_0805_2012Metric")
     )
     (path "/8f77faa8-2d4a-4750-9ffd-4f5c63ff8509/3c0cfff3-c2a3-4531-b7d9-c4df2d10a515"
@@
     )
     (path "/8f77faa8-2d4a-4750-9ffd-4f5c63ff8509/94f4eb33-44aa-4270-b4ae-66e3f7650165"
-      (reference "C47") (unit 1) (value "4u7") (footprint "")
+      (reference "C47") (unit 1) (value "4u7") (footprint "Capacitor_SMD:C_0805_2012Metric")
     )
     (path "/8f77faa8-2d4a-4750-9ffd-4f5c63ff8509/20a7e6cb-cba4-4aff-adbc-921f2e64d818"
@@
     )
     (path "/8f77faa8-2d4a-4750-9ffd-4f5c63ff8509/1a8e78ff-3ba9-48ba-8540-55aaa41723a3"
-      (reference "C49") (unit 1) (value "4u7") (footprint "")
+      (reference "C49") (unit 1) (value "4u7") (footprint "Capacitor_SMD:C_0805_2012Metric")
     )
     (path "/7e318d42-3e09-4c30-96bb-0dfed0f758b6/04b5be4b-63cc-489a-9fb7-b504550ad8f6"
@@
       (reference "D28") (unit 1) (value "RED") (footprint "LED_SMD:LED_0805_2012Metric")
     )
+    (path "/8f77faa8-2d4a-4750-9ffd-4f5c63ff8509/6a1bfc92-66f6-4f98-ba6f-3baefc7c9e1a"
+      (reference "D29") (unit 1) (value "100V") (footprint "")
+    )
     (path "/8f77faa8-2d4a-4750-9ffd-4f5c63ff8509/497a26da-8b1e-4bb2-bcf1-f7f1ed65cd77/75796d65-ffad-48be-a475-bcc6a290f59d"
       (reference "D32") (unit 1) (value "~") (footprint "Diode_SMD:D_SOD-323")
@@
       (reference "Q17") (unit 1) (value "~") (footprint "Package_TO_SOT_SMD:SOT-23")
     )
+    (path "/8f77faa8-2d4a-4750-9ffd-4f5c63ff8509/1612d31f-7850-484e-adc5-384b6ef5aabb"
+      (reference "Q18") (unit 1) (value "BST82,215") (footprint "Package_TO_SOT_SMD:SOT-23")
+    )
     (path "/c2178e99-796d-43c6-a02e-728f26cbf556"
       (reference "R1") (unit 1) (value "5k1") (footprint "Resistor_SMD:R_0805_2012Metric")
@@
       (reference "R63") (unit 1) (value "56") (footprint "Resistor_SMD:R_0805_2012Metric")
     )
+    (path "/8f77faa8-2d4a-4750-9ffd-4f5c63ff8509/7d18e184-9a4b-4d6d-b833-c9b7ccee176f"
+      (reference "R64") (unit 1) (value "100k") (footprint "Resistor_SMD:R_0805_2012Metric")
+    )
+    (path "/8f77faa8-2d4a-4750-9ffd-4f5c63ff8509/403b0429-bf2f-4ddf-af02-08d078bd831c"
+      (reference "R65") (unit 1) (value "1k") (footprint "Resistor_SMD:R_0805_2012Metric")
+    )
+    (path "/8f77faa8-2d4a-4750-9ffd-4f5c63ff8509/46ea8222-b5f0-4bad-9022-155069f4a5a5"
+      (reference "R66") (unit 1) (value "100k") (footprint "Resistor_SMD:R_0805_2012Metric")
+    )
     (path "/8f77faa8-2d4a-4750-9ffd-4f5c63ff8509/497a26da-8b1e-4bb2-bcf1-f7f1ed65cd77/c07ed123-590f-4faa-aa1c-dd5e4f4b12e1"
       (reference "R70") (unit 1) (value "1k") (footprint "Resistor_SMD:R_0805_2012Metric")
@@
     )
     (path "/8f77faa8-2d4a-4750-9ffd-4f5c63ff8509/e40e363c-6474-463d-bcd4-1baf32862bcf"
-      (reference "R78") (unit 1) (value "1k") (footprint "")
+      (reference "R78") (unit 1) (value "1k") (footprint "Resistor_SMD:R_0805_2012Metric")
     )
     (path "/8f77faa8-2d4a-4750-9ffd-4f5c63ff8509/3167b972-519a-4756-9430-dd58932401e5"
@@
     )
     (path "/8f77faa8-2d4a-4750-9ffd-4f5c63ff8509/546ceb14-8790-4e8e-b4cd-895f54381577"
-      (reference "R80") (unit 1) (value "10k") (footprint "")
+      (reference "R80") (unit 1) (value "10k") (footprint "Resistor_SMD:R_0805_2012Metric")
     )
     (path "/8f77faa8-2d4a-4750-9ffd-4f5c63ff8509/701e72b7-fa7f-4613-b62d-5b5bc1923fc6"
-      (reference "R81") (unit 1) (value "10k") (footprint "")
+      (reference "R81") (unit 1) (value "10k") (footprint "Resistor_SMD:R_0805_2012Metric")
     )
     (path "/8f77faa8-2d4a-4750-9ffd-4f5c63ff8509/260d93b6-3321-42fa-9f68-74b7dd975c73"
-      (reference "R82") (unit 1) (value "10k") (footprint "")
+      (reference "R82") (unit 1) (value "10k") (footprint "Resistor_SMD:R_0805_2012Metric")
     )
     (path "/7e318d42-3e09-4c30-96bb-0dfed0f758b6/7eff2d45-424d-41fb-b8b2-85e0be9a1f8b"
@@
       (reference "U5") (unit 1) (value "TJA1051T-3") (footprint "Package_SO:SOIC-8_3.9x4.9mm_P1.27mm")
     )
+    (path "/6d355b13-4b1d-4ba8-891a-0edb0f7a1420"
+      (reference "U6") (unit 1) (value "USBLC6-2SC6") (footprint "Package_TO_SOT_SMD:SOT-23-6")
+    )
     (path "/7e318d42-3e09-4c30-96bb-0dfed0f758b6/580a9e2f-134c-478d-a946-21e4b8d1f45b"

Commit message: almost ready to order
Parts:
- added J8: Conn_01x02, Connector_PinHeader_2.54mm:PinHeader_1x02_P2.54mm_Vertical, symbol Connector_Generic:Conn_01x02
- J3: LCSC C2927038 -> (none)
- J4: footprint Connector_JST:JST_PH_B2B-PH-K_1x02_P2.00mm_Vertical -> Connector_JST:JST_PH_B4B-PH-K_1x04_P2.00mm_Vertical; symbol Connector_Generic:Conn_01x02 -> Connector_Generic:Conn_01x04
Connections:
- net CAN/CAN_H: now also J4.3 (Pin_3); no longer J4.1 (Pin_1)
- net GND: now also J4.1 (Pin_1)
- net STM32L476/USB_DM renamed STM32L476/USB_DN
- new net +5V: J4.4 (Pin_4)
- new net BQ76940/BQ_SCL: J8.1 (Pin_1)
- new net BQ76940/BQ_SDA: J8.2 (Pin_2)
Other:
- sheet BQ76940 ports: added BQ_ALERT, BQ_SCL, BQ_SDA; removed LTC_CS, LTC_SCK, LTC_SDI, LTC_SDO
- sheet Charge_control ports: added CHARGER_CUR, CHARGER_V; removed none
- sheet STM32L476 ports: added BQ_ALERT, BQ_SCL, BQ_SDA, CHARGER_CUR, CHARGER_V, USB_DN; removed CURRENT_MEASURE_EN, LTC_CS, LTC_SCK, LTC_SDI, LTC_SDO, USB_DM

Commit message: V0.2
Parts:
- removed J1, J2: Conn_01x02, Connector_AMASS:AMASS_XT60-M_1x02_P7.20mm_Vertical, symbol Connector_Generic:Conn_01x02
- added NT3: NetTie_2, NetTie:NetTie-2_SMD_Pad2.0mm, symbol Device:NetTie_2
- R1, R2: LCSC (none) -> C27834
- TP1: value TestPoint -> Battery +
- TP2: value TestPoint -> Battery -
Connections:
- net GND: now also NT3.1; no longer TP2.1
- net V+ renamed BAT+
- new net BAT-: NT3.2, TP2.1
Other:
- sheet BQ76940 ports: added BQ_BOOT; removed none
- sheet STM32L476 ports: added BQ_BOOT; removed none
- moved on the sheet: TP1, TP2
