File: LM5164.kicad_sch (KiCad schematic)
At the start: 11 parts, among them U8 ME6118A33

Commit message: before meeting
Parts:
- C50: value (none) -> 2n2; footprint (none) -> Capacitor_SMD:C_0805_2012Metric
- C52: value (none) -> 2u2/100V; footprint (none) -> Capacitor_SMD:C_1206_3216Metric
- C53: value (none) -> 22u; footprint (none) -> Capacitor_SMD:C_1210_3225Metric
- C54, C55: value (none) -> 10u; footprint (none) -> Capacitor_SMD:C_0805_2012Metric
- U9: value (none) -> LM5164DDA; footprint (none) -> Package_SO:HSOP-8-1EP_3.9x4.9mm_P1.27mm_EP2.41x3.1mm_ThermalVias
Changed lines of the file:
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@@
     (in_bom yes) (on_board yes)
     (property "Reference" "C50" (id 0) (at 82.55 45.72 90))
-    (property "Value" "" (id 1) (at 82.55 50.8 90))
-    (property "Footprint" "" (id 2) (at 82.55 47.2948 0)
+    (property "Value" "2n2" (id 1) (at 82.55 50.8 90))
+    (property "Footprint" "Capacitor_SMD:C_0805_2012Metric" (id 2) (at 82.55 47.2948 0)
       (effects (font (size 1.27 1.27)) hide)
     )
@@
     (in_bom yes) (on_board yes) (fields_autoplaced)
     (property "Reference" "U9" (id 0) (at 59.69 40.64 0))
-    (property "Value" "" (id 1) (at 59.69 43.18 0))
-    (property "Footprint" "" (id 2) (at 60.96 67.31 0)
+    (property "Value" "LM5164DDA" (id 1) (at 59.69 43.18 0))
+    (property "Footprint" "Package_SO:HSOP-8-1EP_3.9x4.9mm_P1.27mm_EP2.41x3.1mm_ThermalVias" (id 2) (at 60.96 67.31 0)
       (effects (font (size 1.27 1.27)) hide)
     )
@@
       (effects (font (size 1.27 1.27)) (justify left))
     )
-    (property "Value" "" (id 1) (at 115.57 59.6899 0)
-      (effects (font (size 1.27 1.27)) (justify left))
-    )
-    (property "Footprint" "" (id 2) (at 112.7252 62.23 0)
+    (property "Value" "22u" (id 1) (at 115.57 59.6899 0)
+      (effects (font (size 1.27 1.27)) (justify left))
+    )
+    (property "Footprint" "Capacitor_SMD:C_1210_3225Metric" (id 2) (at 112.7252 62.23 0)
       (effects (font (size 1.27 1.27)) hide)
     )
@@
       (effects (font (size 1.27 1.27)) (justify left))
     )
-    (property "Value" "" (id 1) (at 73.66 116.8399 0)
-      (effects (font (size 1.27 1.27)) (justify left))
-    )
-    (property "Footprint" "" (id 2) (at 70.8152 119.38 0)
+    (property "Value" "10u" (id 1) (at 73.66 116.8399 0)
+      (effects (font (size 1.27 1.27)) (justify left))
+    )
+    (property "Footprint" "Capacitor_SMD:C_0805_2012Metric" (id 2) (at 70.8152 119.38 0)
       (effects (font (size 1.27 1.27)) hide)
     )
@@
       (effects (font (size 1.27 1.27)) (justify left))
     )
-    (property "Value" "" (id 1) (at 34.29 55.8799 0)
-      (effects (font (size 1.27 1.27)) (justify left))
-    )
-    (property "Footprint" "" (id 2) (at 31.4452 58.42 0)
+    (property "Value" "2u2/100V" (id 1) (at 34.29 55.8799 0)
+      (effects (font (size 1.27 1.27)) (justify left))
+    )
+    (property "Footprint" "Capacitor_SMD:C_1206_3216Metric" (id 2) (at 31.4452 58.42 0)
       (effects (font (size 1.27 1.27)) hide)
     )
@@
       (effects (font (size 1.27 1.27)) (justify left))
     )
-    (property "Value" "" (id 1) (at 34.29 116.84 0)
-      (effects (font (size 1.27 1.27)) (justify left))
-    )
-    (property "Footprint" "" (id 2) (at 42.8752 119.38 0)
-      (effects (font (size 1.27 1.27)) hide)
-    )
+    (property "Value" "10u" (id 1) (at 34.29 116.84 0)
+      (effects (font (size 1.27 1.27)) (justify left))
+    )
+    (property "Footprint" "Capacitor_SMD:C_0805_2012Metric" (id 2) (at 42.8752 119.38 0)
+      (effects (font (size 1.27 1.27)) hide)
+    )

Commit message: almost ready to order
Parts:
- added C35: 1n2, Capacitor_SMD:C_0603_1608Metric, symbol Device:C
- added C36: 22u, Capacitor_SMD:C_0805_2012Metric, symbol Device:C
- added C37: 47p, Capacitor_SMD:C_0805_2012Metric, symbol Device:C
- added R67: 237k, Resistor_SMD:R_0805_2012Metric, symbol Device:R
- C50: footprint Capacitor_SMD:C_0805_2012Metric -> Capacitor_SMD:C_0603_1608Metric
- C53: footprint Capacitor_SMD:C_1210_3225Metric -> Capacitor_SMD:C_0805_2012Metric
- L2: value 33u -> 68u; LCSC C206300 -> C206245
- R83: value 316k -> 453k
- R84: value 101k -> 49k9; LCSC C114540 -> (none)
- R85: value 41k2 -> 100k
Connections:
- net +5V: now also C35.2, C36.1
- net FB: now also C37.1
- net GND: now also C36.2
- net SW: now also R67.1
- new net: C35.1, C37.2, R67.2
Other:
- moved on the sheet: C50, C52, C53, L2, R83, R84, R85, U9

Commit message: before switching to kicad 7
Parts:
- C35: LCSC (none) -> C30615
- C36, C53: LCSC C309062 -> C45783
- C37: LCSC (none) -> C14857
- C50: LCSC (none) -> C16033
- C54, C55: LCSC C17024 -> C2932476
- R67: LCSC (none) -> C416833
- R84: LCSC (none) -> C17719
- R85: LCSC (none) -> C149504
Other:
- note added: "Foute waarden"

Commit message: V0.2
Parts:
- C35: value 1n2 -> 2n2; LCSC C30615 -> C1604
- C37: value 47p -> 56p; LCSC C14857 -> C14857
- C50: LCSC C16033 -> C1604
- C54, C55: LCSC C2932476 -> C440198
- L2: value 68u -> 33u; LCSC C206245 -> (none)
- R67: value 237k -> 240k
- R83: value 453k -> 316k
- R84: value 49k9 -> 101k
- R85: value 100k -> 41k2
Connections:
- net V+ renamed BAT+
Other:
- note removed: "300kHz"
- note removed: "Foute waarden"
