File: STM32L476.kicad_sch (KiCad schematic)
At the start: 15 parts, among them U2 STM32L476RGTx, X1 8MHz(16pF)

Commit message: Added part of power schematic
Connections:
- net LTC_CS: now reaches U2.20 (PA4)
- net LTC_SCK: now reaches U2.21 (PA5)
- net LTC_SDO: now reaches U2.22 (PA6)
- net LTC_SDI: now reaches U2.23 (PA7)
- net BQ_PMON_EN: now reaches U2.30 (PB11)
- net BQ_PCHG_EN: now reaches U2.33 (PB12)
- net BQ_CP_EN: now reaches U2.34 (PB13)
- net BQ_DSG_EN: now reaches U2.35 (PB14)
- net BQ_CHG_EN: now reaches U2.36 (PB15)
- net CAN_RX: now reaches U2.61 (PB8)
- net CAN_TX: now reaches U2.62 (PB9)
- net VDD renamed +3V3
Changed lines of the file:
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@@
+    (stroke (width 0) (type default) (color 0 0 0 0))
+  )
+  (wire (pts (xy 152.4 73.66) (xy 154.94 73.66))
     (stroke (width 0) (type default) (color 0 0 0 0))
   )
@@
     (stroke (width 0) (type default) (color 0 0 0 0))
   )
+  (wire (pts (xy 152.4 71.12) (xy 154.94 71.12))
+    (stroke (width 0) (type default) (color 0 0 0 0))
+  )
   (wire (pts (xy 106.68 168.91) (xy 118.11 168.91))
     (stroke (width 0) (type default) (color 0 0 0 0))
@@
     (stroke (width 0) (type default) (color 0 0 0 0))
   )
-  (global_label "LED_RED" (shape input) (at 245.11 59.69 90) (fields_autoplaced)
-    (effects (font (size 1.27 1.27)) (justify left))
-    (property "Intersheet References" "${INTERSHEET_REFS}" (id 0) (at 245.0306 49.1731 90)
-      (effects (font (size 1.27 1.27)) (justify left) hide)
-    )
-  )
-  (global_label "LED_GREEN" (shape input) (at 257.81 59.69 90) (fields_autoplaced)
-    (effects (font (size 1.27 1.27)) (justify left))
-    (property "Intersheet References" "${INTERSHEET_REFS}" (id 0) (at 257.7306 46.6936 90)
-      (effects (font (size 1.27 1.27)) (justify left) hide)
-    )
+  (label "LED_GREEN" (at 257.81 59.69 0)
+    (effects (font (size 1.27 1.27)) (justify left bottom))
+  )
+  (label "LED_RED" (at 245.11 59.69 0)
+    (effects (font (size 1.27 1.27)) (justify left bottom))
+  )
+  (label "LED_GREEN" (at 154.94 73.66 0)
+    (effects (font (size 1.27 1.27)) (justify left bottom))
+  )
+  (label "LED_RED" (at 154.94 71.12 0)
+    (effects (font (size 1.27 1.27)) (justify left bottom))
   )
   (global_label "PH0" (shape input) (at 31.75 78.74 180) (fields_autoplaced)
@@
     )
   )
-  (global_label "LED_RED" (shape input) (at 152.4 71.12 0) (fields_autoplaced)
-    (effects (font (size 1.27 1.27)) (justify left))
-    (property "Intersheet References" "${INTERSHEET_REFS}" (id 0) (at 162.9169 71.0406 0)
-      (effects (font (size 1.27 1.27)) (justify left) hide)
-    )
-  )
   (global_label "PH1" (shape input) (at 116.84 81.28 180) (fields_autoplaced)
     (effects (font (size 1.27 1.27)) (justify right))
@@
     )
   )
-  (global_label "LED_GREEN" (shape input) (at 152.4 73.66 0) (fields_autoplaced)
-    (effects (font (size 1.27 1.27)) (justify left))
-    (property "Intersheet References" "${INTERSHEET_REFS}" (id 0) (at 165.3964 73.5806 0)
-      (effects (font (size 1.27 1.27)) (justify left) hide)
-    )
+  (hierarchical_label "BQ_PMON_EN" (shape input) (at 152.4 119.38 0)
+    (effects (font (size 1.27 1.27)) (justify left))
+  )
+  (hierarchical_label "BQ_DSG_EN" (shape input) (at 152.4 127 0)
+    (effects (font (size 1.27 1.27)) (justify left))
+  )
+  (hierarchical_label "LTC_CS" (shape input) (at 152.4 58.42 0)
+    (effects (font (size 1.27 1.27)) (justify left))
+  )
+  (hierarchical_label "CAN_RX" (shape input) (at 152.4 111.76 0)
+    (effects (font (size 1.27 1.27)) (justify left))
+  )
+  (hierarchical_label "LTC_SDI" (shape input) (at 152.4 66.04 0)
+    (effects (font (size 1.27 1.27)) (justify left))
+  )
+  (hierarchical_label "LTC_SCK" (shape input) (at 152.4 60.96 0)
+    (effects (font (size 1.27 1.27)) (justify left))
+  )
+  (hierarchical_label "BQ_CP_EN" (shape input) (at 152.4 124.46 0)
+    (effects (font (size 1.27 1.27)) (justify left))
+  )
+  (hierarchical_label "BQ_CHG_EN" (shape input) (at 152.4 129.54 0)
+    (effects (font (size 1.27 1.27)) (justify left))
+  )
+  (hierarchical_label "BQ_PCHG_EN" (shape input) (at 152.4 121.92 0)
+    (effects (font (size 1.27 1.27)) (justify left))
+  )
+  (hierarchical_label "LTC_SDO" (shape input) (at 152.4 63.5 0)
+    (effects (font (size 1.27 1.27)) (justify left))
+  )
+  (hierarchical_label "CAN_TX" (shape input) (at 152.4 114.3 0)
+    (effects (font (size 1.27 1.27)) (justify left))
   )
   (symbol (lib_id "Device:Crystal") (at 43.18 78.74 180) (unit 1)
@@
     (pin "1")
   )
-  (symbol (lib_id "power:VDD") (at 45.72 156.21 0) (unit 1)
-    (in_bom yes) (on_board yes) (fields_autoplaced)
-    (property "Reference" "#PWR0110" (id 0) (at 45.72 160.02 0)
-      (effects (font (size 1.27 1.27)) hide)
-    )
-    (property "Value" "VDD" (id 1) (at 45.72 151.13 0))
-    (property "Footprint" "" (id 2) (at 45.72 156.21 0)
-      (effects (font (size 1.27 1.27)) hide)
-    )
-    (property "Datasheet" "" (id 3) (at 45.72 156.21 0)
-      (effects (font (size 1.27 1.27)) hide)
-    )
-    (pin "1")
-  )
   (symbol (lib_id "power:GND") (at 139.7 138.43 0) (unit 1)
     (in_bom yes) (on_board yes) (fields_autoplaced)
@@
     (pin "1")
   )
-  (symbol (lib_id "power:VDD") (at 129.54 40.64 0) (unit 1)
-    (in_bom yes) (on_board yes) (fields_autoplaced)
-    (property "Reference" "#PWR0103" (id 0) (at 129.54 44.45 0)
-      (effects (font (size 1.27 1.27)) hide)
-    )
-    (property "Value" "VDD" (id 1) (at 129.54 35.56 0))
-    (property "Footprint" "" (id 2) (at 129.54 40.64 0)
-      (effects (font (size 1.27 1.27)) hide)
-    )
-    (property "Datasheet" "" (id 3) (at 129.54 40.64 0)
-      (effects (font (size 1.27 1.27)) hide)
-    )
-    (pin "1")
-  )
   (symbol (lib_id "Device:C") (at 80.01 163.83 0) (unit 1)
     (in_bom yes) (on_board yes) (fields_autoplaced)
@@
     )
     (property "Datasheet" "" (id 3) (at 45.72 171.45 0)
+      (effects (font (size 1.27 1.27)) hide)
+    )
+    (pin "1")
+  )
+  (symbol (lib_id "power:+3V3") (at 45.72 156.21 0) (unit 1)
+    (in_bom yes) (on_board yes) (fields_autoplaced)
+    (property "Reference" "#PWR0110" (id 0) (at 45.72 160.02 0)
+      (effects (font (size 1.27 1.27)) hide)
+    )
+    (property "Value" "+3V3" (id 1) (at 45.72 151.13 0))
+    (property "Footprint" "" (id 2) (at 45.72 156.21 0)
+      (effects (font (size 1.27 1.27)) hide)
+    )
+    (property "Datasheet" "" (id 3) (at 45.72 156.21 0)
       (effects (font (size 1.27 1.27)) hide)
     )
@@
       (effects (font (size 1.27 1.27)) hide)
     )
+    (pin "1")
+  )
+  (symbol (lib_id "power:+3V3") (at 129.54 40.64 0) (unit 1)
+    (in_bom yes) (on_board yes) (fields_autoplaced)
+    (property "Reference" "#PWR0103" (id 0) (at 129.54 44.45 0)
+      (effects (font (size 1.27 1.27)) hide)
+    )
+    (property "Value" "+3V3" (id 1) (at 129.54 35.56 0))
+    (property "Footprint" "" (id 2) (at 129.54 40.64 0)
+      (effects (font (size 1.27 1.27)) hide)
+    )
+    (property "Datasheet" "" (id 3) (at 129.54 40.64 0)
+      (effects (font (size 1.27 1.27)) hide)
+    )

Commit message: update
Parts:
- X1: footprint Crystal:Crystal_SMD_2012-2Pin_2.0x1.2mm -> Crystal:Crystal_SMD_5032-2Pin_5.0x3.2mm
Connections:
- net USB_DM: now reaches U2.44 (PA11)
- net USB_DP: now reaches U2.45 (PA12)
- net CURRENT_MEASURE_EN: now reaches U2.58 (PB6)
Changed lines of the file:
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@@
+    (effects (font (size 1.27 1.27)) (justify left))
+  )
+  (hierarchical_label "USB_DP" (shape input) (at 152.4 78.74 0)
     (effects (font (size 1.27 1.27)) (justify left))
   )
@@
     (effects (font (size 1.27 1.27)) (justify left))
   )
+  (hierarchical_label "CURRENT_MEASURE_EN" (shape input) (at 152.4 106.68 0)
+    (effects (font (size 1.27 1.27)) (justify left))
+  )
   (hierarchical_label "LTC_SCK" (shape input) (at 152.4 60.96 0)
+    (effects (font (size 1.27 1.27)) (justify left))
+  )
+  (hierarchical_label "USB_DM" (shape input) (at 152.4 76.2 0)
     (effects (font (size 1.27 1.27)) (justify left))
   )
@@
     (property "Reference" "X1" (id 0) (at 43.18 71.12 0))
     (property "Value" "8MHz(16pF)" (id 1) (at 43.18 73.66 0))
-    (property "Footprint" "Crystal:Crystal_SMD_2012-2Pin_2.0x1.2mm" (id 2) (at 43.18 78.74 0)
+    (property "Footprint" "Crystal:Crystal_SMD_5032-2Pin_5.0x3.2mm" (id 2) (at 43.18 78.74 0)
       (effects (font (size 1.27 1.27)) hide)
     )

Commit message: routed most tracks
Parts:
- added C46: C, symbol Device:C
- added J7: Conn_01x05, Connector_JST:JST_PH_B5B-PH-K_1x05_P2.00mm_Vertical, symbol Connector_Generic:Conn_01x05
Connections:
- net +3V3: now also J7.1 (Pin_1)
- net GND: now also C46.2, J7.5 (Pin_5)
- net SWCLK: now reaches U2.46 (PA13)
- net SWCLK: now also J7.3 (Pin_3)
- net SWDIO: now reaches U2.49 (PA14)
- net SWDIO: now also J7.4 (Pin_4)
- net NRST: now reaches U2.7 (NRST)
- net NRST: now also C46.1, J7.2 (Pin_2)
- no-connect marks 2 -> 1
Other:
- moved on the sheet: C13, C14, C15, C16, C17, C18, C19, C20, C21, X1

Commit message: new board dimensions
Parts:
- C14: renamed from C46; footprint (none) -> Capacitor_SMD:C_0805_2012Metric
- U2: LCSC (none) -> C92468; Remark (none) -> STM32L431 for now
- renumbered C13 to C15, C15 to C16, C20 to C17, C21 to C18, C14 to C19, C16 to C20, C17 to C21, C18 to C22, C19 to C23, D1 to D25, D2 to D26, R37 to R51, R38 to R52
Changed lines of the file:
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@@
   (symbol (lib_id "power:GND") (at 257.81 85.09 0) (unit 1)
     (in_bom yes) (on_board yes) (fields_autoplaced)
-    (property "Reference" "#PWR0106" (id 0) (at 257.81 91.44 0)
+    (property "Reference" "#PWR012" (id 0) (at 257.81 91.44 0)
       (effects (font (size 1.27 1.27)) hide)
     )
@@
   (symbol (lib_id "Device:LED") (at 245.11 77.47 90) (unit 1)
     (in_bom yes) (on_board yes) (fields_autoplaced)
-    (property "Reference" "D1" (id 0) (at 248.92 77.7874 90)
+    (property "Reference" "D25" (id 0) (at 248.92 77.7874 90)
       (effects (font (size 1.27 1.27)) (justify right))
     )
@@
   (symbol (lib_id "power:GND") (at 95.25 166.37 0) (unit 1)
     (in_bom yes) (on_board yes) (fields_autoplaced)
-    (property "Reference" "#PWR0107" (id 0) (at 95.25 172.72 0)
+    (property "Reference" "#PWR019" (id 0) (at 95.25 172.72 0)
       (effects (font (size 1.27 1.27)) hide)
     )
@@
   (symbol (lib_id "power:GND") (at 139.7 138.43 0) (unit 1)
     (in_bom yes) (on_board yes) (fields_autoplaced)
-    (property "Reference" "#PWR0102" (id 0) (at 139.7 144.78 0)
+    (property "Reference" "#PWR016" (id 0) (at 139.7 144.78 0)
       (effects (font (size 1.27 1.27)) hide)
     )
@@
   (symbol (lib_id "power:GND") (at 134.62 138.43 0) (unit 1)
     (in_bom yes) (on_board yes) (fields_autoplaced)
-    (property "Reference" "#PWR0101" (id 0) (at 134.62 144.78 0)
+    (property "Reference" "#PWR015" (id 0) (at 134.62 144.78 0)
       (effects (font (size 1.27 1.27)) hide)
     )
@@
   (symbol (lib_id "Device:C") (at 68.58 160.02 0) (unit 1)
     (in_bom yes) (on_board yes) (fields_autoplaced)
-    (property "Reference" "C18" (id 0) (at 72.39 158.7499 0)
+    (property "Reference" "C22" (id 0) (at 72.39 158.7499 0)
       (effects (font (size 1.27 1.27)) (justify left))
     )
@@
   (symbol (lib_id "power:GND") (at 34.29 167.64 0) (unit 1)
     (in_bom yes) (on_board yes) (fields_autoplaced)
-    (property "Reference" "#PWR0109" (id 0) (at 34.29 173.99 0)
+    (property "Reference" "#PWR020" (id 0) (at 34.29 173.99 0)
       (effects (font (size 1.27 1.27)) hide)
     )
@@
   (symbol (lib_id "power:+3V3") (at 34.29 152.4 0) (unit 1)
     (in_bom yes) (on_board yes) (fields_autoplaced)
-    (property "Reference" "#PWR0110" (id 0) (at 34.29 156.21 0)
+    (property "Reference" "#PWR018" (id 0) (at 34.29 156.21 0)
       (effects (font (size 1.27 1.27)) hide)
     )
@@
   (symbol (lib_id "Device:C") (at 57.15 160.02 0) (unit 1)
     (in_bom yes) (on_board yes) (fields_autoplaced)
-    (property "Reference" "C17" (id 0) (at 60.96 158.7499 0)
+    (property "Reference" "C21" (id 0) (at 60.96 158.7499 0)
       (effects (font (size 1.27 1.27)) (justify left))
     )
@@
   (symbol (lib_id "Device:C") (at 50.8 99.06 0) (unit 1)
     (in_bom yes) (on_board yes) (fields_autoplaced)
-    (property "Reference" "C15" (id 0) (at 54.61 97.7899 0)
+    (property "Reference" "C16" (id 0) (at 54.61 97.7899 0)
       (effects (font (size 1.27 1.27)) (justify left))
     )
@@
   (symbol (lib_id "Device:R") (at 257.81 67.31 0) (unit 1)
     (in_bom yes) (on_board yes) (fields_autoplaced)
-    (property "Reference" "R38" (id 0) (at 260.35 66.0399 0)
+    (property "Reference" "R52" (id 0) (at 260.35 66.0399 0)
       (effects (font (size 1.27 1.27)) (justify left))
     )
@@
     )
     (property "Datasheet" "http://www.st.com/st-web-ui/static/active/en/resource/technical/document/datasheet/DM00108832.pdf" (id 3) (at 134.62 88.9 0)
+      (effects (font (size 1.27 1.27)) hide)
+    )
+    (property "LCSC" "C92468" (id 4) (at 134.62 88.9 0)
+      (effects (font (size 1.27 1.27)) hide)
+    )
+    (property "Remark" "STM32L431 for now" (id 5) (at 134.62 88.9 0)
       (effects (font (size 1.27 1.27)) hide)
     )
@@
   (symbol (lib_id "Device:R") (at 245.11 67.31 0) (unit 1)
     (in_bom yes) (on_board yes) (fields_autoplaced)
-    (property "Reference" "R37" (id 0) (at 247.65 66.0399 0)
+    (property "Reference" "R51" (id 0) (at 247.65 66.0399 0)
       (effects (font (size 1.27 1.27)) (justify left))
     )
@@
   (symbol (lib_id "power:GND") (at 105.41 58.42 0) (unit 1)
     (in_bom yes) (on_board yes) (fields_autoplaced)
-    (property "Reference" "#PWR0136" (id 0) (at 105.41 64.77 0)
+    (property "Reference" "#PWR09" (id 0) (at 105.41 64.77 0)
       (effects (font (size 1.27 1.27)) hide)
     )
@@
   (symbol (lib_id "Device:C") (at 35.56 99.06 0) (unit 1)
     (in_bom yes) (on_board yes) (fields_autoplaced)
-    (property "Reference" "C13" (id 0) (at 39.37 97.7899 0)
+    (property "Reference" "C15" (id 0) (at 39.37 97.7899 0)
       (effects (font (size 1.27 1.27)) (justify left))
     )
@@
   (symbol (lib_id "Device:C") (at 45.72 160.02 0) (unit 1)
     (in_bom yes) (on_board yes) (fields_autoplaced)
-    (property "Reference" "C16" (id 0) (at 49.53 158.7499 0)
+    (property "Reference" "C20" (id 0) (at 49.53 158.7499 0)
       (effects (font (size 1.27 1.27)) (justify left))
     )
@@
   (symbol (lib_id "Device:C") (at 106.68 158.75 0) (unit 1)
     (in_bom yes) (on_board yes) (fields_autoplaced)
-    (property "Reference" "C21" (id 0) (at 110.49 157.4799 0)
+    (property "Reference" "C18" (id 0) (at 110.49 157.4799 0)
       (effects (font (size 1.27 1.27)) (justify left))
     )
@@
   (symbol (lib_id "power:GND") (at 245.11 85.09 0) (unit 1)
     (in_bom yes) (on_board yes) (fields_autoplaced)
-    (property "Reference" "#PWR0105" (id 0) (at 245.11 91.44 0)
+    (property "Reference" "#PWR011" (id 0) (at 245.11 91.44 0)
       (effects (font (size 1.27 1.27)) hide)
     )
@@
   (symbol (lib_id "Device:C") (at 95.25 158.75 0) (unit 1)
     (in_bom yes) (on_board yes) (fields_autoplaced)
-    (property "Reference" "C20" (id 0) (at 99.06 157.4799 0)
+    (property "Reference" "C17" (id 0) (at 99.06 157.4799 0)
       (effects (font (size 1.27 1.27)) (justify left))
     )
@@
   (symbol (lib_id "Device:C") (at 80.01 160.02 0) (unit 1)
     (in_bom yes) (on_board yes) (fields_autoplaced)
-    (property "Reference" "C19" (id 0) (at 83.82 158.7499 0)
+    (property "Reference" "C23" (id 0) (at 83.82 158.7499 0)
       (effects (font (size 1.27 1.27)) (justify left))
     )
@@
   (symbol (lib_id "power:GND") (at 35.56 104.14 0) (unit 1)
     (in_bom yes) (on_board yes) (fields_autoplaced)
-    (property "Reference" "#PWR0111" (id 0) (at 35.56 110.49 0)
+    (property "Reference" "#PWR013" (id 0) (at 35.56 110.49 0)
       (effects (font (size 1.27 1.27)) hide)
     )
@@
   (symbol (lib_id "Device:LED") (at 257.81 77.47 90) (unit 1)
     (in_bom yes) (on_board yes) (fields_autoplaced)
-    (property "Reference" "D2" (id 0) (at 261.62 77.7874 90)
+    (property "Reference" "D26" (id 0) (at 261.62 77.7874 90)
       (effects (font (size 1.27 1.27)) (justify right))
     )
@@
   (symbol (lib_id "power:VDDA") (at 95.25 151.13 0) (unit 1)
     (in_bom yes) (on_board yes) (fields_autoplaced)
-    (property "Reference" "#PWR0108" (id 0) (at 95.25 154.94 0)
+    (property "Reference" "#PWR017" (id 0) (at 95.25 154.94 0)
       (effects (font (size 1.27 1.27)) hide)
     )
@@
   (symbol (lib_id "power:+3V3") (at 129.54 40.64 0) (unit 1)
     (in_bom yes) (on_board yes) (fields_autoplaced)
-    (property "Reference" "#PWR0103" (id 0) (at 129.54 44.45 0)
+    (property "Reference" "#PWR06" (id 0) (at 129.54 44.45 0)
       (effects (font (size 1.27 1.27)) hide)
     )
@@
   (symbol (lib_id "power:GND") (at 45.72 59.69 0) (unit 1)
     (in_bom yes) (on_board yes) (fields_autoplaced)
-    (property "Reference" "#PWR0135" (id 0) (at 45.72 66.04 0)
+    (property "Reference" "#PWR010" (id 0) (at 45.72 66.04 0)
       (effects (font (size 1.27 1.27)) hide)
     )
@@
   (symbol (lib_id "power:+3V3") (at 45.72 43.18 0) (unit 1)
     (in_bom yes) (on_board yes) (fields_autoplaced)
-    (property "Reference" "#PWR0134" (id 0) (at 45.72 46.99 0)
+    (property "Reference" "#PWR08" (id 0) (at 45.72 46.99 0)
       (effects (font (size 1.27 1.27)) hide)
     )
@@
   (symbol (lib_id "Device:C") (at 34.29 160.02 0) (unit 1)
     (in_bom yes) (on_board yes) (fields_autoplaced)
-    (property "Reference" "C14" (id 0) (at 38.1 158.7499 0)
+    (property "Reference" "C19" (id 0) (at 38.1 158.7499 0)
       (effects (font (size 1.27 1.27)) (justify left))
     )
@@
   (symbol (lib_id "power:VDDA") (at 139.7 40.64 0) (unit 1)
     (in_bom yes) (on_board yes) (fields_autoplaced)
-    (property "Reference" "#PWR0104" (id 0) (at 139.7 44.45 0)
+    (property "Reference" "#PWR07" (id 0) (at 139.7 44.45 0)
       (effects (font (size 1.27 1.27)) hide)
     )
@@
   (symbol (lib_id "Device:C") (at 105.41 53.34 0) (unit 1)
     (in_bom yes) (on_board yes) (fields_autoplaced)
-    (property "Reference" "C46" (id 0) (at 109.22 52.0699 0)
+    (property "Reference" "C14" (id 0) (at 109.22 52.0699 0)
       (effects (font (size 1.27 1.27)) (justify left))
     )
@@
       (effects (font (size 1.27 1.27)) (justify left))
     )
-    (property "Footprint" "" (id 2) (at 106.3752 57.15 0)
+    (property "Footprint" "Capacitor_SMD:C_0805_2012Metric" (id 2) (at 106.3752 57.15 0)
       (effects (font (size 1.27 1.27)) hide)
     )
@@
   (symbol (lib_id "power:GND") (at 50.8 104.14 0) (unit 1)
     (in_bom yes) (on_board yes) (fields_autoplaced)
-    (property "Reference" "#PWR0112" (id 0) (at 50.8 110.49 0)
-      (effects (font (size 1.27 1.27)) hide)
-    )
+    (property "Reference" "#PWR014" (id 0) (at 50.8 110.49 0)
+      (effects (font (size 1.27 1.27)) hide)
+    )

Commit message: almost ready to order
Parts:
- removed X1: 8MHz(16pF), Crystal:Crystal_SMD_5032-2Pin_5.0x3.2mm, symbol Device:Crystal
- added Y1: 8Mhz, Crystal:Crystal_SMD_3225-4Pin_3.2x2.5mm, symbol Device:Crystal_GND24
- C14: value C -> 100n; footprint Capacitor_SMD:C_0805_2012Metric -> Capacitor_SMD:C_0603_1608Metric
- C15, C16: value 20p -> 15p; footprint Capacitor_SMD:C_0805_2012Metric -> Capacitor_SMD:C_0603_1608Metric
- C17, C18, C19, C20, C21, C22: footprint Capacitor_SMD:C_0805_2012Metric -> Capacitor_SMD:C_0603_1608Metric
- C23: value 4,7u -> 4u7; footprint Capacitor_SMD:C_0805_2012Metric -> Capacitor_SMD:C_0603_1608Metric
- R51, R52: value 100 -> 220
Connections:
- net LTC_SDI is gone; now on net BQ_DSG_EN: U2.23 (PA7)
- net LTC_SDO is gone; now on net BQ_PMON_EN: U2.22 (PA6)
- net +3V3: now also J7.5 (Pin_5); no longer J7.1 (Pin_1)
- net BQ_CHG_EN: now also U2.25 (PC5); no longer U2.36 (PB15)
- net BQ_CP_EN: now also U2.24 (PC4); no longer U2.34 (PB13)
- net BQ_DSG_EN: no longer U2.35 (PB14)
- net BQ_PMON_EN: no longer U2.30 (PB11)
- net GND: now also J7.3 (Pin_3), U2.60 (BOOT0), Y1.2, Y1.4; no longer J7.5 (Pin_5)
- net LED_GREEN: now also U2.16 (PA2); no longer U2.43 (PA10)
- net LED_RED: now also U2.15 (PA1); no longer U2.42 (PA9)
- net NRST: now also J7.1 (Pin_1); no longer J7.2 (Pin_2)
- net PH0: now also Y1.1
- net PH1: now also Y1.3
- net SWCLK: now also J7.4 (Pin_4), U2.49 (PA14); no longer J7.3 (Pin_3), U2.46 (PA13)
- net SWDIO: now also J7.2 (Pin_2), U2.46 (PA13); no longer J7.4 (Pin_4), U2.49 (PA14)
- net CHARGER_CUR: now reaches U2.11 (PC3)
- net CHARGER_V: now reaches U2.26 (PB0)
- net BQ_SCL: now reaches U2.29 (PB10)
- net BQ_PCHG_EN: no longer names the net of U2.33 (PB12)
- net CURRENT_MEASURE_EN: no longer names the net of U2.58 (PB6)
- net LTC_CS: no longer names the net of U2.20 (PA4)
- net LTC_SCK: no longer names the net of U2.21 (PA5)
- net USB_DM renamed USB_DN
- new net BQ_ALERT: U2.36 (PB15)
- new net BQ_SDA: U2.30 (PB11)
- no-connect marks 1 -> 23
Other:
- moved on the sheet: C14, C15, C16
