File: STM32L476.kicad_sch (KiCad schematic)
At the start: 17 parts, among them J7 Conn_01x05, U2 STM32L476RGTx, Y1 8Mhz

Commit message: before switching to kicad 7
Parts:
- C14, C17, C19, C20, C21, C22: LCSC (none) -> C1591
- C15, C16: LCSC (none) -> C1644
- C18: LCSC (none) -> C5673
- C23: LCSC (none) -> C69335
- D25: LCSC (none) -> C84256
- R51, R52: LCSC (none) -> C17557
Changed lines of the file:
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@@
+      (effects (font (size 1.27 1.27)) hide)
+    )
+    (property "LCSC" "C84256" (id 4) (at 245.11 77.47 0)
       (effects (font (size 1.27 1.27)) hide)
     )
@@
       (effects (font (size 1.27 1.27)) hide)
     )
+    (property "LCSC" "C1591" (id 4) (at 68.58 160.02 0)
+      (effects (font (size 1.27 1.27)) hide)
+    )
     (pin "1")
     (pin "2")
@@
       (effects (font (size 1.27 1.27)) hide)
     )
+    (property "LCSC" "C1591" (id 4) (at 57.15 160.02 0)
+      (effects (font (size 1.27 1.27)) hide)
+    )
     (pin "1")
     (pin "2")
@@
       (effects (font (size 1.27 1.27)) hide)
     )
+    (property "LCSC" "C1644" (id 4) (at 53.34 99.06 0)
+      (effects (font (size 1.27 1.27)) hide)
+    )
     (pin "1")
     (pin "2")
@@
     )
     (property "Datasheet" "~" (id 3) (at 257.81 67.31 0)
+      (effects (font (size 1.27 1.27)) hide)
+    )
+    (property "LCSC" "C17557" (id 4) (at 257.81 67.31 0)
       (effects (font (size 1.27 1.27)) hide)
     )
@@
       (effects (font (size 1.27 1.27)) hide)
     )
+    (property "LCSC" "C17557" (id 4) (at 245.11 67.31 0)
+      (effects (font (size 1.27 1.27)) hide)
+    )
     (pin "1")
     (pin "2")
@@
       (effects (font (size 1.27 1.27)) hide)
     )
-    (property "LCSC" "" (id 4) (at 30.48 99.06 0)
+    (property "LCSC" "C1644" (id 4) (at 30.48 99.06 0)
       (effects (font (size 1.27 1.27)) hide)
     )
@@
       (effects (font (size 1.27 1.27)) hide)
     )
+    (property "LCSC" "C1591" (id 4) (at 45.72 160.02 0)
+      (effects (font (size 1.27 1.27)) hide)
+    )
     (pin "1")
     (pin "2")
@@
       (effects (font (size 1.27 1.27)) hide)
     )
+    (property "LCSC" "C5673" (id 4) (at 106.68 158.75 0)
+      (effects (font (size 1.27 1.27)) hide)
+    )
     (pin "1")
     (pin "2")
@@
       (effects (font (size 1.27 1.27)) hide)
     )
+    (property "LCSC" "C1591" (id 4) (at 95.25 158.75 0)
+      (effects (font (size 1.27 1.27)) hide)
+    )
     (pin "1")
     (pin "2")
@@
     )
     (property "Datasheet" "~" (id 3) (at 80.01 160.02 0)
+      (effects (font (size 1.27 1.27)) hide)
+    )
+    (property "LCSC" "C69335" (id 4) (at 80.01 160.02 0)
       (effects (font (size 1.27 1.27)) hide)
     )
@@
       (effects (font (size 1.27 1.27)) hide)
     )
+    (property "LCSC" "C1591" (id 4) (at 34.29 160.02 0)
+      (effects (font (size 1.27 1.27)) hide)
+    )
     (pin "1")
     (pin "2")
@@
       (effects (font (size 1.27 1.27)) hide)
     )
+    (property "LCSC" "C1591" (id 4) (at 97.79 53.34 0)
+      (effects (font (size 1.27 1.27)) hide)
+    )

Commit message: V0.2
Parts:
- C14, C17, C19, C20, C21, C22: LCSC C1591 -> C14663
- C18: LCSC C5673 -> C15849
- C23: LCSC C69335 -> C19666
- D26: LCSC (none) -> C84256
Connections:
- net BQ_BOOT: now reaches U2.27 (PB1)
- no-connect marks 23 -> 22
